File: Schematics/74HC138 Test/74HC138Test.sch (KiCad schematic (older format))
At the start: 22 parts, among them U1 74HC138

Commit message: Minor fixes in 74HC138 test schematic
Parts:
- added C?: 100 nF, symbol C
Connections:
- wire segments 54 -> 58
Changed lines of the file:
@@
 LIBS:valves
 LIBS:74xgxx
+LIBS:74HC138Test-cache
 EELAYER 25 0
 EELAYER END
@@
 P 6000 4300
 F 0 "U1" H 6100 4800 50  0000 C CNN
-F 1 "74HC138" H 6150 3751 50  0000 C CNN
+F 1 "74HC138" H 6200 3750 50  0000 C CNN
 F 2 "" H 6000 4300 50  0001 C CNN
 F 3 "" H 6000 4300 50  0001 C CNN
@@
 Connection ~ 4650 4150
 Wire Wire Line
-	3800 3250 4650 3250
+	3800 3250 6000 3250
 Connection ~ 4550 3250
 Connection ~ 3800 3250
@@
 Text Label 8200 7650 0    60   ~ 0
 26/11/2017
+Wire Wire Line
+	6000 3250 6000 3850
+Connection ~ 4650 3250
+Wire Wire Line
+	6000 4750 6000 5100
+Connection ~ 6000 5100
+$Comp
+L C C?
+U 1 1 5A2CE301
+P 5400 3500
+F 0 "C?" H 5425 3600 50  0001 L CNN
+F 1 "100 nF" H 5425 3400 50  0000 L CNN
+F 2 "" H 5438 3350 50  0001 C CNN
+F 3 "" H 5400 3500 50  0001 C CNN
+	1    5400 3500
+	1    0    0    -1
+$EndComp
+Wire Wire Line
+	5400 3350 5400 3250
+Connection ~ 5400 3250
+$Comp
+L GND #PWR?
+U 1 1 5A2CE3B9
+P 5400 3750
+F 0 "#PWR?" H 5400 3500 50  0001 C CNN
+F 1 "GND" H 5400 3600 50  0000 C CNN
+F 2 "" H 5400 3750 50  0001 C CNN
+F 3 "" H 5400 3750 50  0001 C CNN
+	1    5400 3750
+	1    0    0    -1
+$EndComp
+Wire Wire Line
+	5400 3650 5400 3750
 $EndSCHEMATC

Commit message: Update schematics to KiCad 5
Parts:
- C?: symbol CP -> Device:CP
- C?: symbol C -> Device:C
- D? (x8): symbol LED -> Device:LED
- R1, R? (x10): symbol R -> Device:R
- SW?: symbol SW_DIP_x03 -> switches:SW_DIP_x03
- U1: symbol 74LS138 -> 74HC138Test-rescue:74LS138
Connections:
- wire segments 58 -> 80
Changed lines of the file:
@@
-EESchema Schematic File Version 2
-LIBS:power
-LIBS:device
-LIBS:switches
-LIBS:relays
-LIBS:motors
-LIBS:transistors
-LIBS:conn
-LIBS:linear
-LIBS:regul
-LIBS:74xx
-LIBS:cmos4000
-LIBS:adc-dac
-LIBS:memory
-LIBS:xilinx
-LIBS:microcontrollers
-LIBS:dsp
-LIBS:microchip
-LIBS:analog_switches
-LIBS:motorola
-LIBS:texas
-LIBS:intel
-LIBS:audio
-LIBS:interface
-LIBS:digital-audio
-LIBS:philips
-LIBS:display
-LIBS:cypress
-LIBS:siliconi
-LIBS:opto
-LIBS:atmel
-LIBS:contrib
-LIBS:valves
-LIBS:74xgxx
+EESchema Schematic File Version 4
 LIBS:74HC138Test-cache
-EELAYER 25 0
+EELAYER 26 0
 EELAYER END
 $Descr A4 11693 8268
@@
 $EndDescr
 $Comp
-L GND #PWR?
+L power:GND #PWR?
 U 1 1 5A1A81EB
 P 3800 5100
@@
 $EndComp
 $Comp
-L VCC #PWR?
+L power:VCC #PWR?
 U 1 1 5A1A8201
 P 3800 3100
@@
 $EndComp
 $Comp
-L SW_DIP_x03 SW?
+L switches:SW_DIP_x03 SW?
 U 1 1 5A1A828F
 P 4450 3550
@@
 $EndComp
 $Comp
-L R R1
+L Device:R R1
 U 1 1 5A1A84D8
 P 4450 4350
@@
 $EndComp
 $Comp
-L R R?
+L Device:R R?
 U 1 1 5A1A8569
 P 4550 4350
@@
 $EndComp
 $Comp
-L R R?
+L Device:R R?
 U 1 1 5A1A8577
 P 4650 4350
@@
 $EndComp
 $Comp
-L R R?
+L Device:R R?
 U 1 1 5A1A8853
 P 6850 3950
@@
 $EndComp
 $Comp
-L R R?
+L Device:R R?
 U 1 1 5A1A88F9
 P 6850 4050
@@
 $EndComp
 $Comp
-L R R?
+L Device:R R?
 U 1 1 5A1A8907
 P 6850 4150
@@
 $EndComp
 $Comp
-L R R?
+L Device:R R?
 U 1 1 5A1A8915
 P 6850 4250
@@
 $EndComp
 $Comp
-L R R?
+L Device:R R?
 U 1 1 5A1A8923
 P 6850 4350
@@
 $EndComp
 $Comp
-L R R?
+L Device:R R?
 U 1 1 5A1A8931
 P 6850 4450
@@
 $EndComp
 $Comp
-L R R?
+L Device:R R?
 U 1 1 5A1A8940
 P 6850 4550
@@
 $EndComp
 $Comp
-L R R?
+L Device:R R?
 U 1 1 5A1A8950
 P 6850 4650
@@
 $EndComp
 $Comp
-L LED D?
+L Device:LED D?
 U 1 1 5A1A8A88
 P 7500 3950
@@
 $EndComp
 $Comp
-L LED D?
+L Device:LED D?
 U 1 1 5A1A8AD8
 P 7500 4100
@@
 $EndComp
 $Comp
-L LED D?
+L Device:LED D?
 U 1 1 5A1A8AF6
 P 7500 4250
@@
 $EndComp
 $Comp
-L LED D?
+L Device:LED D?
 U 1 1 5A1A8B04
 P 7500 4400
@@
 $EndComp
 $Comp
-L LED D?
+L Device:LED D?
 U 1 1 5A1A8B12
 P 7500 4550
@@
 $EndComp
 $Comp
-L LED D?
+L Device:LED D?
 U 1 1 5A1A8B20
 P 7500 4700
@@
 $EndComp
 $Comp
-L LED D?
+L Device:LED D?
 U 1 1 5A1A8B2E
 P 7500 4850
@@
 $EndComp
 $Comp
-L LED D?
+L Device:LED D?
 U 1 1 5A1A8B3C
 P 7500 5000
@@
 $EndComp
 $Comp
-L 74LS138 U1
+L 74HC138Test-rescue:74LS138 U1
 U 1 1 5A1A814D
 P 6000 4300
@@
 $EndComp
 Wire Wire Line
-	3800 3100 3800 4650
-Wire Wire Line
-	4450 3850 4450 4200
-Wire Wire Line
-	4550 3850 4550 4200
-Wire Wire Line
-	4650 3850 4650 4200
+	3800 3100 3800 3250
+Wire Wire Line
+	4450 3850 4450 3950
+Wire Wire Line
+	4550 3850 4550 4050
+Wire Wire Line
+	4650 3850 4650 4150
 Wire Wire Line
 	5350 4450 5400 4450
@@
 Connection ~ 4650 4150
 Wire Wire Line
-	3800 3250 6000 3250
+	3800 3250 4450 3250
 Connection ~ 4550 3250
 Connection ~ 3800 3250
@@
 	7650 3950 7850 3950
 Wire Wire Line
-	7850 3950 7850 5100
+	7850 3950 7850 4100
 Wire Wire Line
 	7850 4100 7650 4100
@@
 Connection ~ 7850 5000
 Wire Wire Line
-	7850 5100 3800 5100
-Wire Wire Line
-	5400 4550 5400 5100
+	7850 5100 6000 5100
+Wire Wire Line
+	5400 4550 5400 4650
 Connection ~ 5400 5100
 Connection ~ 5400 4650
@@
 	5350 4550 3800 4550
 $Comp
-L CP C?
+L Device:CP C?
 U 1 1 5A1A9453
 P 3800 4800
@@
 Connection ~ 6000 5100
 $Comp
-L C C?
+L Device:C C?
 U 1 1 5A2CE301
 P 5400 3500
@@
 Connection ~ 5400 3250
 $Comp
-L GND #PWR?
+L power:GND #PWR?
 U 1 1 5A2CE3B9
 P 5400 3750
@@
 Wire Wire Line
 	5400 3650 5400 3750
+Wire Wire Line
+	4450 3950 4450 4200
+Wire Wire Line
+	4550 4050 4550 4200
+Wire Wire Line
+	4650 4150 4650 4200
+Wire Wire Line
+	4550 3250 4650 3250
+Wire Wire Line
+	3800 3250 3800 4550
+Wire Wire Line
+	4450 3250 4550 3250
+Wire Wire Line
+	7850 4100 7850 4250
+Wire Wire Line
+	7850 4250 7850 4400
+Wire Wire Line
+	7850 4400 7850 4550
+Wire Wire Line
+	7850 4550 7850 4700
+Wire Wire Line
+	7850 4700 7850 4850
+Wire Wire Line
+	7850 4850 7850 5000
+Wire Wire Line
+	7850 5000 7850 5100
+Wire Wire Line
+	5400 5100 4650 5100
+Wire Wire Line
+	5400 4650 5400 5100
+Wire Wire Line
+	4650 5100 4550 5100
+Wire Wire Line
+	4550 5100 4450 5100
+Wire Wire Line
+	4450 5100 3800 5100
+Wire Wire Line
+	3800 4550 3800 4650
+Wire Wire Line
+	4650 3250 5400 3250
+Wire Wire Line
+	6000 5100 5400 5100
+Wire Wire Line
+	5400 3250 6000 3250
 $EndSCHEMATC

Commit message: Save all Schematics again to overcome problems with version change
Parts:
- SW?: symbol switches:SW_DIP_x03 -> 74HC138Test-rescue:SW_DIP_x03-switches
Changed lines of the file:
@@
 $EndComp
 $Comp
-L switches:SW_DIP_x03 SW?
+L 74HC138Test-rescue:SW_DIP_x03-switches SW?
 U 1 1 5A1A828F
 P 4450 3550
