File: Schematics/Address Bus Spy/AddressBusSpy.sch (KiCad schematic (older format))
At the start: 38 parts, among them U1 74HC00, U2 74HCT244

Commit message: Add PCB for Address Bus Spy schematic
Parts:
- removed C1: 1uF, symbol CP
- added C4: 100nF, Capacitors_THT:C_Disc_D10.0mm_W2.5mm_P5.00mm, symbol C_Small
- added J1: Conn_01x20, Pin_Headers:Pin_Header_Straight_1x20_Pitch2.54mm, symbol Conn_01x20
- A0, A1, A10, A11, A12, A13, A14, A15, A2, A3, A4, A5, A6, A7, A8, A9: footprint (none) -> RainbowLibrary:LED_thickpad
- C2, C3: footprint (none) -> Capacitors_THT:C_Disc_D10.0mm_W2.5mm_P5.00mm
- R1, R10, R11, R12, R13, R14, R15, R16, R2, R3, R4, R5, R6, R7, R8, R9: renamed from R?; footprint (none) -> RainbowLibrary:R_Axial_DIN0204_L3.6mm_D1.6mm_P7.62mm_Horizontal
- U1: renamed from U?; footprint (none) -> RainbowLibrary:DIP-20_thickpad
- U2: footprint (none) -> RainbowLibrary:DIP-20_thickpad
- U3: renamed from U1; footprint (none) -> RainbowLibrary:DIP-14_thickpad
Connections:
- wire segments 139 -> 201
Other:
- note added: "1.1"
- note removed: "1.00"

Commit message: Update schematics to KiCad 5
Parts:
- A0, A1, A10, A11, A12, A13, A14, A15, A2, A3, A4, A5, A6, A7, A8, A9: symbol LED -> Device:LED
- C2, C3, C4: symbol C_Small -> Device:C_Small
- J1: symbol Conn_01x20 -> conn:Conn_01x20
- R1, R10, R11, R12, R13, R14, R15, R16, R2, R3, R4, R5, R6, R7, R8, R9: symbol R -> Device:R
- U1, U2: symbol 74HCT244 -> AddressBusSpy-rescue:74HCT244
- U3: symbol 74HC00 -> AddressBusSpy-rescue:74HC00
Connections:
- wire segments 201 -> 243

Commit message: Save all Schematics again to overcome problems with version change
Parts:
- J1: symbol conn:Conn_01x20 -> AddressBusSpy-rescue:Conn_01x20-conn
Changed lines of the file:
@@
 $EndComp
 $Comp
-L conn:Conn_01x20 J1
+L AddressBusSpy-rescue:Conn_01x20-conn J1
 U 1 1 5A34884C
 P 2250 5200
