File: Schematics/Address Decoder/AddressDecoder.sch (KiCad schematic (older format))
At the start: 3 parts, among them U1 Atmel 28C64, U2 74HCT138, U3 6116

Commit message: Update schematics to KiCad 5
Parts:
- U1: symbol 27C64 -> memory:27C64
- U2: symbol 74LS138 -> AddressDecoder-rescue:74LS138
- U3: symbol 6116 -> memory:6116
Connections:
- wire segments 76 -> 86
Changed lines of the file:
@@
-EESchema Schematic File Version 2
-LIBS:power
-LIBS:device
-LIBS:switches
-LIBS:relays
-LIBS:motors
-LIBS:transistors
-LIBS:conn
-LIBS:linear
-LIBS:regul
-LIBS:74xx
-LIBS:cmos4000
-LIBS:adc-dac
-LIBS:memory
-LIBS:xilinx
-LIBS:microcontrollers
-LIBS:dsp
-LIBS:microchip
-LIBS:analog_switches
-LIBS:motorola
-LIBS:texas
-LIBS:intel
-LIBS:audio
-LIBS:interface
-LIBS:digital-audio
-LIBS:philips
-LIBS:display
-LIBS:cypress
-LIBS:siliconi
-LIBS:opto
-LIBS:atmel
-LIBS:contrib
-LIBS:valves
-LIBS:Zilog
+EESchema Schematic File Version 4
 LIBS:AddressDecoder-cache
-EELAYER 25 0
+EELAYER 26 0
 EELAYER END
 $Descr A4 11693 8268
@@
 $EndDescr
 $Comp
-L 6116 U3
+L memory:6116 U3
 U 1 1 5A2E5CEB
 P 6950 4600
@@
 $EndComp
 $Comp
-L VCC #PWR?
+L power:VCC #PWR?
 U 1 1 5A2E60EC
 P 3950 1050
@@
 1.0
 $Comp
-L GND #PWR?
+L power:GND #PWR?
 U 1 1 5A2E6C9B
 P 3950 5550
@@
 Z80_ADDRESS_BUS
 $Comp
-L 27C64 U1
+L memory:27C64 U1
 U 1 1 5A2E5C26
 P 6950 2450
@@
 	6950 1250 6950 1500
 Wire Wire Line
-	3950 1050 3950 3000
+	3950 1050 3950 1250
 Wire Wire Line
 	6950 3850 6950 3700
@@
 Connection ~ 6950 1250
 Wire Wire Line
-	8750 1250 2950 1250
+	8750 1250 6950 1250
 Connection ~ 3950 1250
 Wire Wire Line
 	6950 5500 6950 5350
 Wire Wire Line
-	3950 3900 3950 5550
-Wire Wire Line
-	3200 5500 6950 5500
+	3950 3900 3950 5500
+Wire Wire Line
+	3200 5500 3350 5500
 Connection ~ 3950 5500
 Wire Wire Line
@@
 	3350 3200 3200 3200
 Wire Wire Line
-	3200 3200 3200 5500
+	3200 3200 3200 3300
 Wire Wire Line
 	3200 3300 3350 3300
@@
 	3350 3700 2400 3700
 Wire Wire Line
-	5250 2600 5250 5100
+	5250 2600 5250 3350
 Wire Wire Line
 	5250 3350 6250 3350
@@
 	5250 5100 6350 5100
 Connection ~ 5250 3350
-Wire Bus Line
-	8250 4800 8250 1400
 Entry Bus Bus
 	8150 1550 8250 1650
@@
 	7550 4600 8150 4600
 Wire Bus Line
-	5950 1400 5950 4950
-Wire Bus Line
 	5950 1400 5150 1400
 Entry Bus Bus
@@
 	6050 4900 6350 4900
 $Comp
-L 74LS138 U2
+L AddressDecoder-rescue:74LS138 U2
 U 1 1 5A2E603E
 P 3950 3450
@@
 Wire Wire Line
 	3250 3400 2400 3400
+Wire Wire Line
+	6950 1250 5650 1250
+Wire Wire Line
+	3950 1250 3950 3000
+Wire Wire Line
+	3950 1250 2950 1250
+Wire Wire Line
+	3950 5500 3950 5550
+Wire Wire Line
+	3950 5500 5450 5500
+Wire Wire Line
+	5450 5500 6950 5500
+Wire Wire Line
+	3350 5500 3950 5500
+Wire Wire Line
+	3200 3300 3200 5500
+Wire Wire Line
+	5250 3350 5250 5100
+Wire Wire Line
+	5650 1250 3950 1250
+Wire Bus Line
+	8250 1400 8250 4800
+Wire Bus Line
+	5950 1400 5950 4950
 $EndSCHEMATC

Commit message: Save all Schematics again to overcome problems with version change
Parts:
- U1: symbol memory:27C64 -> AddressDecoder-rescue:27C64-memory
- U3: symbol memory:6116 -> AddressDecoder-rescue:6116-memory
Changed lines of the file:
@@
 $EndDescr
 $Comp
-L memory:6116 U3
+L AddressDecoder-rescue:6116-memory U3
 U 1 1 5A2E5CEB
 P 6950 4600
@@
 Z80_ADDRESS_BUS
 $Comp
-L memory:27C64 U1
+L AddressDecoder-rescue:27C64-memory U1
 U 1 1 5A2E5C26
 P 6950 2450
