File: Schematics/ControlBusLEDs/ControlBusLEDs.sch (KiCad schematic (older format))
At the start: 18 parts, among them J1 Conn_02x08_Top_Bottom, M1 LED_ALT, U2 74HC240

Commit message: Minor nits in control bus LEDs schematic
Connections:
- net labels added: GND, VCC
- wire segments 90 -> 89
Changed lines of the file:
@@
 Connection ~ 7750 4750
 Connection ~ 7750 5000
-Wire Wire Line
-	7750 3250 7750 5800
 $Comp
 L Conn_02x08_Top_Bottom J1
@@
 P 3050 4600
 F 0 "J1" H 3100 5000 50  0000 C CNN
-F 1 "Conn_02x08_Top_Bottom" H 3300 4050 50  0000 C CNN
+F 1 "Conn_02x08_Top_Bottom" H 3300 4050 50  0001 C CNN
 F 2 "Connectors_Multicomp:Multicomp_MC9A12-1634_2x08x2.54mm_Straight" H 3050 4600 50  0001 C CNN
 F 3 "" H 3050 4600 50  0001 C CNN
@@
 $EndComp
 Wire Wire Line
-	7750 5800 4800 5800
-Wire Wire Line
-	4800 5800 4800 5500
-Wire Wire Line
-	4800 3700 4800 4100
+	4800 3550 4800 4100
 Wire Wire Line
 	4300 5200 4300 5600
 Connection ~ 4300 5300
 Wire Wire Line
-	3600 5600 4800 5600
-Connection ~ 4800 5600
+	7750 5600 3600 5600
 Wire Wire Line
-	3600 5600 3600 4900
+	3600 4900 3600 5800
 Wire Wire Line
 	3600 4900 3350 4900
@@
 Wire Wire Line
 	2500 4600 2850 4600
+Wire Wire Line
+	4800 5600 4800 5500
+Wire Wire Line
+	7750 3250 7750 5600
+Connection ~ 4800 5600
+$Comp
+L VCC #PWR?
+U 1 1 5A2D11F3
+P 4800 3550
+F 0 "#PWR?" H 4800 3400 50  0001 C CNN
+F 1 "VCC" H 4800 3700 50  0000 C CNN
+F 2 "" H 4800 3550 50  0001 C CNN
+F 3 "" H 4800 3550 50  0001 C CNN
+	1    4800 3550
+	1    0    0    -1
+$EndComp
+$Comp
+L GND #PWR?
+U 1 1 5A2D128B
+P 3600 5800
+F 0 "#PWR?" H 3600 5550 50  0001 C CNN
+F 1 "GND" H 3600 5650 50  0000 C CNN
+F 2 "" H 3600 5800 50  0001 C CNN
+F 3 "" H 3600 5800 50  0001 C CNN
+	1    3600 5800
+	1    0    0    -1
+$EndComp
+Connection ~ 3600 5600
 $EndSCHEMATC

Commit message: Remove connector from ControlBusLEDs schematic. Add .gitignore
Parts:
- removed J1: Conn_02x08_Top_Bottom, Connectors_Multicomp:Multicomp_MC9A12-1634_2x08x2.54mm_Straight, symbol Conn_02x08_Top_Bottom
Connections:
- net labels added: ~BUSACK, ~BUSRQ, ~HALT, ~IORQ, ~M1, ~MREQ, ~RD, ~WR
- wire segments 89 -> 75
Other:
- note added: "1.01"
- note added: "11/12/17"
Changed lines of the file:
@@
 	0    -1   -1   0
 $EndComp
-Wire Wire Line
-	5300 5000 5650 5000
-Wire Wire Line
-	5300 4900 5650 4900
-Wire Wire Line
-	5650 4900 5650 4850
-Wire Wire Line
-	5300 4800 5650 4800
-Wire Wire Line
-	5650 4800 5650 4700
-Wire Wire Line
-	5300 4700 5600 4700
-Wire Wire Line
-	5600 4700 5600 4550
-Wire Wire Line
-	5600 4550 5650 4550
-Wire Wire Line
-	5300 4600 5550 4600
-Wire Wire Line
-	5550 4600 5550 4400
-Wire Wire Line
-	5550 4400 5650 4400
-Wire Wire Line
-	5300 4500 5500 4500
-Wire Wire Line
-	5500 4500 5500 4250
-Wire Wire Line
-	5500 4250 5650 4250
-Wire Wire Line
-	5300 4400 5450 4400
-Wire Wire Line
-	5450 4400 5450 4100
-Wire Wire Line
-	5450 4100 5650 4100
-Wire Wire Line
-	5300 4300 5400 4300
-Wire Wire Line
-	5400 4300 5400 3950
-Wire Wire Line
-	5400 3950 5650 3950
 $Comp
 L LED_ALT M1
@@
 	-1   0    0    1
 $EndComp
-Wire Wire Line
-	5950 5000 7050 5000
-Wire Wire Line
-	5950 4850 7050 4850
-Wire Wire Line
-	7050 4850 7050 4750
-Wire Wire Line
-	5950 4700 7050 4700
-Wire Wire Line
-	7050 4700 7050 4500
-Wire Wire Line
-	5950 4550 6950 4550
-Wire Wire Line
-	6950 4550 6950 4250
-Wire Wire Line
-	6950 4250 7050 4250
-Wire Wire Line
-	5950 4400 6850 4400
-Wire Wire Line
-	6850 4400 6850 4000
-Wire Wire Line
-	6850 4000 7050 4000
-Wire Wire Line
-	5950 4250 6750 4250
-Wire Wire Line
-	6750 4250 6750 3750
-Wire Wire Line
-	6750 3750 7050 3750
-Wire Wire Line
-	5950 4100 6650 4100
-Wire Wire Line
-	6650 4100 6650 3500
-Wire Wire Line
-	6650 3500 7050 3500
-Wire Wire Line
-	5950 3950 6550 3950
-Wire Wire Line
-	6550 3950 6550 3250
-Wire Wire Line
-	6550 3250 7050 3250
-Wire Wire Line
-	7350 3250 7750 3250
-Wire Wire Line
-	7750 3500 7350 3500
-Wire Wire Line
-	7750 3750 7350 3750
-Connection ~ 7750 3500
-Wire Wire Line
-	7750 4000 7350 4000
-Connection ~ 7750 3750
-Wire Wire Line
-	7750 4250 7350 4250
-Connection ~ 7750 4000
-Wire Wire Line
-	7750 4500 7350 4500
-Connection ~ 7750 4250
-Wire Wire Line
-	7750 4750 7350 4750
-Connection ~ 7750 4500
-Wire Wire Line
-	7750 5000 7350 5000
-Connection ~ 7750 4750
-Connection ~ 7750 5000
-$Comp
-L Conn_02x08_Top_Bottom J1
-U 1 1 5A1D99EC
-P 3050 4600
-F 0 "J1" H 3100 5000 50  0000 C CNN
-F 1 "Conn_02x08_Top_Bottom" H 3300 4050 50  0001 C CNN
-F 2 "Connectors_Multicomp:Multicomp_MC9A12-1634_2x08x2.54mm_Straight" H 3050 4600 50  0001 C CNN
-F 3 "" H 3050 4600 50  0001 C CNN
-	1    3050 4600
-	1    0    0    -1
-$EndComp
-Wire Wire Line
-	4800 3550 4800 4100
-Wire Wire Line
-	4300 5200 4300 5600
-Connection ~ 4300 5300
-Wire Wire Line
-	7750 5600 3600 5600
-Wire Wire Line
-	3600 4900 3600 5800
-Wire Wire Line
-	3600 4900 3350 4900
-Connection ~ 4300 5600
-Wire Wire Line
-	2850 4300 2800 4300
-Wire Wire Line
-	2800 4300 2800 3850
-Wire Wire Line
-	2800 3850 4800 3850
-Connection ~ 4800 3850
-Wire Wire Line
-	4300 4300 3750 4300
-Wire Wire Line
-	3750 4300 3750 3950
-Wire Wire Line
-	3750 3950 2600 3950
-Wire Wire Line
-	2600 3950 2600 4400
-Wire Wire Line
-	3600 4400 3600 4050
-Wire Wire Line
-	3600 4050 2500 4050
-Wire Wire Line
-	2500 4050 2500 4600
-Wire Wire Line
-	3550 4500 3550 3750
-Wire Wire Line
-	3550 3750 2400 3750
-Wire Wire Line
-	2400 3750 2400 4800
-Wire Wire Line
-	2400 4800 2850 4800
-Wire Wire Line
-	4300 4600 3950 4600
-Wire Wire Line
-	3950 4600 3950 3650
-Wire Wire Line
-	3950 3650 2300 3650
-Wire Wire Line
-	2300 3650 2300 5000
-Wire Wire Line
-	2300 5000 2850 5000
-Wire Wire Line
-	3350 4400 3500 4400
-Wire Wire Line
-	3500 4400 3500 5000
-Wire Wire Line
-	3500 5000 4300 5000
-Wire Wire Line
-	3350 4600 3650 4600
-Wire Wire Line
-	3650 4600 3650 4900
-Wire Wire Line
-	3650 4900 4300 4900
-Wire Wire Line
-	3350 4800 4300 4800
-Wire Wire Line
-	3350 5000 3350 5200
-Wire Wire Line
-	3350 5200 4050 5200
-Wire Wire Line
-	4050 5200 4050 4700
-Wire Wire Line
-	4050 4700 4300 4700
-Wire Wire Line
-	4300 4400 3600 4400
-Wire Wire Line
-	4300 4500 3550 4500
-Wire Wire Line
-	2600 4400 2850 4400
-Wire Wire Line
-	2500 4600 2850 4600
-Wire Wire Line
-	4800 5600 4800 5500
-Wire Wire Line
-	7750 3250 7750 5600
-Connection ~ 4800 5600
 $Comp
 L VCC #PWR?
@@
 L GND #PWR?
 U 1 1 5A2D128B
-P 3600 5800
-F 0 "#PWR?" H 3600 5550 50  0001 C CNN
-F 1 "GND" H 3600 5650 50  0000 C CNN
-F 2 "" H 3600 5800 50  0001 C CNN
-F 3 "" H 3600 5800 50  0001 C CNN
-	1    3600 5800
+P 4800 5800
+F 0 "#PWR?" H 4800 5550 50  0001 C CNN
+F 1 "GND" H 4800 5650 50  0000 C CNN
+F 2 "" H 4800 5800 50  0001 C CNN
+F 3 "" H 4800 5800 50  0001 C CNN
+	1    4800 5800
 	1    0    0    -1
 $EndComp
-Connection ~ 3600 5600
+Text GLabel 3450 4200 0    60   Input ~ 0
+~BUSACK
+Text GLabel 3450 4350 0    60   Input ~ 0
+~BUSRQ
+Text GLabel 3450 4500 0    60   Input ~ 0
+~IORQ
+Text GLabel 3450 4650 0    60   Input ~ 0
+~MREQ
+Text GLabel 3450 4800 0    60   Input ~ 0
+~WR
+Text GLabel 3450 4950 0    60   Input ~ 0
+~RD
+Text GLabel 3450 5100 0    60   Input ~ 0
+~HALT
+Text GLabel 3450 5250 0    60   Input ~ 0
+~M1
+Wire Wire Line
+	5300 5000 5650 5000
+Wire Wire Line
+	5300 4900 5650 4900
+Wire Wire Line
+	5650 4900 5650 4850
+Wire Wire Line
+	5300 4800 5650 4800
+Wire Wire Line
+	5650 4800 5650 4700
+Wire Wire Line
+	5300 4700 5600 4700
+Wire Wire Line
+	5600 4700 5600 4550
+Wire Wire Line
+	5600 4550 5650 4550
+Wire Wire Line
+	5300 4600 5550 4600
+Wire Wire Line
+	5550 4600 5550 4400
+Wire Wire Line
+	5550 4400 5650 4400
+Wire Wire Line
+	5300 4500 5500 4500
+Wire Wire Line
+	5500 4500 5500 4250
+Wire Wire Line
+	5500 4250 5650 4250
+Wire Wire Line
+	5300 4400 5450 4400
+Wire Wire Line
+	5450 4400 5450 4100
+Wire Wire Line
+	5450 4100 5650 4100
+Wire Wire Line
+	5300 4300 5400 4300
+Wire Wire Line
+	5400 4300 5400 3950
+Wire Wire Line
+	5400 3950 5650 3950
+Wire Wire Line
+	5950 5000 7050 5000
+Wire Wire Line
+	5950 4850 7050 4850
+Wire Wire Line
+	7050 4850 7050 4750
+Wire Wire Line
+	5950 4700 7050 4700
+Wire Wire Line
+	7050 4700 7050 4500
+Wire Wire Line
+	5950 4550 6950 4550
+Wire Wire Line
+	6950 4550 6950 4250
+Wire Wire Line
+	6950 4250 7050 4250
+Wire Wire Line
+	5950 4400 6850 4400
+Wire Wire Line
+	6850 4400 6850 4000
+Wire Wire Line
+	6850 4000 7050 4000
+Wire Wire Line
+	5950 4250 6750 4250
+Wire Wire Line
+	6750 4250 6750 3750
+Wire Wire Line
+	6750 3750 7050 3750
+Wire Wire Line
+	5950 4100 6650 4100
+Wire Wire Line
+	6650 4100 6650 3500
+Wire Wire Line
+	6650 3500 7050 3500
+Wire Wire Line
+	5950 3950 6550 3950
+Wire Wire Line
+	6550 3950 6550 3250
+Wire Wire Line
+	6550 3250 7050 3250
+Wire Wire Line
+	7350 3250 7750 3250
+Wire Wire Line
+	7750 3500 7350 3500
+Wire Wire Line
+	7750 3750 7350 3750
+Connection ~ 7750 3500
+Wire Wire Line
+	7750 4000 7350 4000
+Connection ~ 7750 3750
+Wire Wire Line
+	7750 4250 7350 4250
+Connection ~ 7750 4000
+Wire Wire Line
+	7750 4500 7350 4500
+Connection ~ 7750 4250
+Wire Wire Line
+	7750 4750 7350 4750
+Connection ~ 7750 4500
+Wire Wire Line
+	7750 5000 7350 5000
+Connection ~ 7750 4750
+Connection ~ 7750 5000
+Wire Wire Line
+	4800 3550 4800 4100
+Wire Wire Line
+	7750 5600 7750 3250
+Wire Wire Line
+	4300 5600 7750 5600
+Wire Wire Line
+	4800 5500 4800 5800
+Connection ~ 4800 5600
+Wire Wire Line
+	3450 4200 4200 4200
+Wire Wire Line
+	4200 4200 4200 4300
+Wire Wire Line
+	4200 4300 4300 4300
+Wire Wire Line
+	3450 4350 4150 4350
+Wire Wire Line
+	4150 4350 4150 4400
+Wire Wire Line
+	4150 4400 4300 4400
+Wire Wire Line
+	3450 4500 4300 4500
+Wire Wire Line
+	3450 4650 4150 4650
+Wire Wire Line
+	4150 4650 4150 4600
+Wire Wire Line
+	4150 4600 4300 4600
+Wire Wire Line
+	3450 4800 4100 4800
+Wire Wire Line
+	4100 4800 4100 4700
+Wire Wire Line
+	4100 4700 4300 4700
+Wire Wire Line
+	3450 4950 4150 4950
+Wire Wire Line
+	4150 4950 4150 4800
+Wire Wire Line
+	4150 4800 4300 4800
+Wire Wire Line
+	3450 5100 4200 5100
+Wire Wire Line
+	4200 5100 4200 4900
+Wire Wire Line
+	4200 4900 4300 4900
+Wire Wire Line
+	3450 5250 4250 5250
+Wire Wire Line
+	4250 5250 4250 5000
+Wire Wire Line
+	4250 5000 4300 5000
+Wire Wire Line
+	4300 5200 4300 5600
+Connection ~ 4300 5300
+Text Notes 8200 7650 0    60   ~ 0
+11/12/17
+Text Notes 10600 7650 0    60   ~ 0
+1.01
 $EndSCHEMATC

Commit message: Update ControlBusLEDs schematic and add initial PCB
Parts:
- added C1: 100 nF, Capacitors_THT:C_Disc_D10.0mm_W2.5mm_P5.00mm, symbol C
- added J1: Conn_01x10, Pin_Headers:Pin_Header_Straight_1x10_Pitch2.54mm, symbol Conn_01x10
Connections:
- wire segments 75 -> 98
Changed lines of the file:
@@
 $EndComp
 $Comp
-L VCC #PWR?
+L VCC #PWR01
 U 1 1 5A2D11F3
 P 4800 3550
-F 0 "#PWR?" H 4800 3400 50  0001 C CNN
+F 0 "#PWR01" H 4800 3400 50  0001 C CNN
 F 1 "VCC" H 4800 3700 50  0000 C CNN
 F 2 "" H 4800 3550 50  0001 C CNN
@@
 $EndComp
 $Comp
-L GND #PWR?
+L GND #PWR02
 U 1 1 5A2D128B
 P 4800 5800
-F 0 "#PWR?" H 4800 5550 50  0001 C CNN
+F 0 "#PWR02" H 4800 5550 50  0001 C CNN
 F 1 "GND" H 4800 5650 50  0000 C CNN
 F 2 "" H 4800 5800 50  0001 C CNN
@@
 	1    0    0    -1
 $EndComp
-Text GLabel 3450 4200 0    60   Input ~ 0
+Text GLabel 3150 4200 0    60   Input ~ 0
 ~BUSACK
-Text GLabel 3450 4350 0    60   Input ~ 0
+Text GLabel 3150 4350 0    60   Input ~ 0
 ~BUSRQ
-Text GLabel 3450 4500 0    60   Input ~ 0
+Text GLabel 3150 4500 0    60   Input ~ 0
 ~IORQ
-Text GLabel 3450 4650 0    60   Input ~ 0
+Text GLabel 3150 4650 0    60   Input ~ 0
 ~MREQ
-Text GLabel 3450 4800 0    60   Input ~ 0
+Text GLabel 3150 4800 0    60   Input ~ 0
 ~WR
-Text GLabel 3450 4950 0    60   Input ~ 0
+Text GLabel 3150 4950 0    60   Input ~ 0
 ~RD
-Text GLabel 3450 5100 0    60   Input ~ 0
+Text GLabel 3150 5100 0    60   Input ~ 0
 ~HALT
-Text GLabel 3450 5250 0    60   Input ~ 0
+Text GLabel 3150 5250 0    60   Input ~ 0
 ~M1
-Wire Wire Line
-	5300 5000 5650 5000
-Wire Wire Line
-	5300 4900 5650 4900
-Wire Wire Line
-	5650 4900 5650 4850
-Wire Wire Line
-	5300 4800 5650 4800
-Wire Wire Line
-	5650 4800 5650 4700
-Wire Wire Line
-	5300 4700 5600 4700
-Wire Wire Line
-	5600 4700 5600 4550
-Wire Wire Line
-	5600 4550 5650 4550
-Wire Wire Line
-	5300 4600 5550 4600
-Wire Wire Line
-	5550 4600 5550 4400
-Wire Wire Line
-	5550 4400 5650 4400
-Wire Wire Line
-	5300 4500 5500 4500
-Wire Wire Line
-	5500 4500 5500 4250
-Wire Wire Line
-	5500 4250 5650 4250
-Wire Wire Line
-	5300 4400 5450 4400
-Wire Wire Line
-	5450 4400 5450 4100
-Wire Wire Line
-	5450 4100 5650 4100
-Wire Wire Line
-	5300 4300 5400 4300
-Wire Wire Line
-	5400 4300 5400 3950
-Wire Wire Line
-	5400 3950 5650 3950
-Wire Wire Line
-	5950 5000 7050 5000
-Wire Wire Line
-	5950 4850 7050 4850
-Wire Wire Line
-	7050 4850 7050 4750
-Wire Wire Line
-	5950 4700 7050 4700
-Wire Wire Line
-	7050 4700 7050 4500
-Wire Wire Line
-	5950 4550 6950 4550
-Wire Wire Line
-	6950 4550 6950 4250
-Wire Wire Line
-	6950 4250 7050 4250
-Wire Wire Line
-	5950 4400 6850 4400
-Wire Wire Line
-	6850 4400 6850 4000
-Wire Wire Line
-	6850 4000 7050 4000
-Wire Wire Line
-	5950 4250 6750 4250
-Wire Wire Line
-	6750 4250 6750 3750
-Wire Wire Line
-	6750 3750 7050 3750
-Wire Wire Line
-	5950 4100 6650 4100
-Wire Wire Line
-	6650 4100 6650 3500
-Wire Wire Line
-	6650 3500 7050 3500
-Wire Wire Line
-	5950 3950 6550 3950
-Wire Wire Line
-	6550 3950 6550 3250
-Wire Wire Line
-	6550 3250 7050 3250
-Wire Wire Line
-	7350 3250 7750 3250
-Wire Wire Line
-	7750 3500 7350 3500
-Wire Wire Line
-	7750 3750 7350 3750
-Connection ~ 7750 3500
-Wire Wire Line
-	7750 4000 7350 4000
-Connection ~ 7750 3750
-Wire Wire Line
-	7750 4250 7350 4250
-Connection ~ 7750 4000
-Wire Wire Line
-	7750 4500 7350 4500
-Connection ~ 7750 4250
-Wire Wire Line
-	7750 4750 7350 4750
-Connection ~ 7750 4500
-Wire Wire Line
-	7750 5000 7350 5000
-Connection ~ 7750 4750
-Connection ~ 7750 5000
-Wire Wire Line
-	4800 3550 4800 4100
-Wire Wire Line
-	7750 5600 7750 3250
-Wire Wire Line
-	4300 5600 7750 5600
-Wire Wire Line
-	4800 5500 4800 5800
-Connection ~ 4800 5600
-Wire Wire Line
-	3450 4200 4200 4200
-Wire Wire Line
-	4200 4200 4200 4300
-Wire Wire Line
-	4200 4300 4300 4300
-Wire Wire Line
-	3450 4350 4150 4350
-Wire Wire Line
-	4150 4350 4150 4400
-Wire Wire Line
-	4150 4400 4300 4400
-Wire Wire Line
-	3450 4500 4300 4500
-Wire Wire Line
-	3450 4650 4150 4650
-Wire Wire Line
-	4150 4650 4150 4600
-Wire Wire Line
-	4150 4600 4300 4600
-Wire Wire Line
-	3450 4800 4100 4800
-Wire Wire Line
-	4100 4800 4100 4700
-Wire Wire Line
-	4100 4700 4300 4700
-Wire Wire Line
-	3450 4950 4150 4950
-Wire Wire Line
-	4150 4950 4150 4800
-Wire Wire Line
-	4150 4800 4300 4800
-Wire Wire Line
-	3450 5100 4200 5100
-Wire Wire Line
-	4200 5100 4200 4900
-Wire Wire Line
-	4200 4900 4300 4900
-Wire Wire Line
-	3450 5250 4250 5250
-Wire Wire Line
-	4250 5250 4250 5000
-Wire Wire Line
-	4250 5000 4300 5000
-Wire Wire Line
-	4300 5200 4300 5600
-Connection ~ 4300 5300
 Text Notes 8200 7650 0    60   ~ 0
 11/12/17
 Text Notes 10600 7650 0    60   ~ 0
 1.01
+$Comp
+L Conn_01x10 J1
+U 1 1 5A324482
+P 2800 3500
+F 0 "J1" H 2800 4000 50  0000 C CNN
+F 1 "Conn_01x10" H 2800 2900 50  0000 C CNN
+F 2 "Pin_Headers:Pin_Header_Straight_1x10_Pitch2.54mm" H 2800 3500 50  0001 C CNN
+F 3 "" H 2800 3500 50  0001 C CNN
+	1    2800 3500
+	-1   0    0    1
+$EndComp
+$Comp
+L C C1
+U 1 1 5A32538A
+P 5150 3800
+F 0 "C1" H 5175 3900 50  0000 L CNN
+F 1 "100 nF" H 5175 3700 50  0000 L CNN
+F 2 "Capacitors_THT:C_Disc_D10.0mm_W2.5mm_P5.00mm" H 5188 3650 50  0001 C CNN
+F 3 "" H 5150 3800 50  0001 C CNN
+	1    5150 3800
+	1    0    0    -1
+$EndComp
+Wire Wire Line
+	5300 5000 5650 5000
+Wire Wire Line
+	5300 4900 5650 4900
+Wire Wire Line
+	5650 4900 5650 4850
+Wire Wire Line
+	5300 4800 5650 4800
+Wire Wire Line
+	5650 4800 5650 4700
+Wire Wire Line
+	5300 4700 5600 4700
+Wire Wire Line
+	5600 4700 5600 4550
+Wire Wire Line
+	5600 4550 5650 4550
+Wire Wire Line
+	5300 4600 5550 4600
+Wire Wire Line
+	5550 4600 5550 4400
+Wire Wire Line
+	5550 4400 5650 4400
+Wire Wire Line
+	5300 4500 5500 4500
+Wire Wire Line
+	5500 4500 5500 4250
+Wire Wire Line
+	5500 4250 5650 4250
+Wire Wire Line
+	5300 4400 5450 4400
+Wire Wire Line
+	5450 4400 5450 4100
+Wire Wire Line
+	5450 4100 5650 4100
+Wire Wire Line
+	5300 4300 5400 4300
+Wire Wire Line
+	5400 4300 5400 3950
+Wire Wire Line
+	5400 3950 5650 3950
+Wire Wire Line
+	5950 5000 7050 5000
+Wire Wire Line
+	5950 4850 7050 4850
+Wire Wire Line
+	7050 4850 7050 4750
+Wire Wire Line
+	5950 4700 7050 4700
+Wire Wire Line
+	7050 4700 7050 4500
+Wire Wire Line
+	5950 4550 6950 4550
+Wire Wire Line
+	6950 4550 6950 4250
+Wire Wire Line
+	6950 4250 7050 4250
+Wire Wire Line
+	5950 4400 6850 4400
+Wire Wire Line
+	6850 4400 6850 4000
+Wire Wire Line
+	6850 4000 7050 4000
+Wire Wire Line
+	5950 4250 6750 4250
+Wire Wire Line
+	6750 4250 6750 3750
+Wire Wire Line
+	6750 3750 7050 3750
+Wire Wire Line
+	5950 4100 6650 4100
+Wire Wire Line
+	6650 4100 6650 3500
+Wire Wire Line
+	6650 3500 7050 3500
+Wire Wire Line
+	5950 3950 6550 3950
+Wire Wire Line
+	6550 3950 6550 3250
+Wire Wire Line
+	6550 3250 7050 3250
+Wire Wire Line
+	7350 3250 7750 3250
+Wire Wire Line
+	7750 3500 7350 3500
+Wire Wire Line
+	7750 3750 7350 3750
+Connection ~ 7750 3500
+Wire Wire Line
+	7750 4000 7350 4000
+Connection ~ 7750 3750
+Wire Wire Line
+	7750 4250 7350 4250
+Connection ~ 7750 4000
+Wire Wire Line
+	7750 4500 7350 4500
+Connection ~ 7750 4250
+Wire Wire Line
+	7750 4750 7350 4750
+Connection ~ 7750 4500
+Wire Wire Line
+	7750 5000 7350 5000
+Connection ~ 7750 4750
+Connection ~ 7750 5000
+Wire Wire Line
+	4800 3550 4800 4100
+Wire Wire Line
+	7750 3250 7750 5600
+Wire Wire Line
+	7750 5600 4100 5600
+Wire Wire Line
+	4800 5500 4800 5800
+Connection ~ 4800 5600
+Wire Wire Line
+	4300 5600 4300 5200
+Connection ~ 4300 5300
+Wire Wire Line
+	3150 4200 4000 4200
+Wire Wire Line
+	4000 4200 4000 4300
+Wire Wire Line
+	4000 4300 4300 4300
+Wire Wire Line
+	3150 4350 3900 4350
+Wire Wire Line
+	3900 4350 3900 4400
+Wire Wire Line
+	3900 4400 4300 4400
+Wire Wire Line
+	3150 4500 4300 4500
+Wire Wire Line
+	3150 4650 3900 4650
+Wire Wire Line
+	3900 4650 3900 4600
+Wire Wire Line
+	3900 4600 4300 4600
+Wire Wire Line
+	3150 4800 3900 4800
+Wire Wire Line
+	3900 4800 3900 4700
+Wire Wire Line
+	3900 4700 4300 4700
+Wire Wire Line
+	3150 4950 4000 4950
+Wire Wire Line
+	4000 4950 4000 4800
+Wire Wire Line
+	4000 4800 4300 4800
+Wire Wire Line
+	3150 5100 4050 5100
+Wire Wire Line
+	4050 5100 4050 4900
+Wire Wire Line
+	4050 4900 4300 4900
+Wire Wire Line
+	3150 5250 4150 5250
+Wire Wire Line
+	4150 5250 4150 5000
+Wire Wire Line
+	4150 5000 4300 5000
+Wire Wire Line
+	3200 3900 3200 5250
+Connection ~ 3200 5250
+Wire Wire Line
+	3000 3800 3300 3800
+Wire Wire Line
+	3300 3800 3300 5100
+Connection ~ 3300 5100
+Wire Wire Line
+	3000 3700 3400 3700
+Wire Wire Line
+	3400 3700 3400 4950
+Connection ~ 3400 4950
+Wire Wire Line
+	3000 3600 3500 3600
+Wire Wire Line
+	3500 3600 3500 4800
+Connection ~ 3500 4800
+Wire Wire Line
+	3000 3500 3600 3500
+Wire Wire Line
+	3600 3500 3600 4650
+Connection ~ 3600 4650
+Wire Wire Line
+	3000 3400 3700 3400
+Wire Wire Line
+	3700 3400 3700 4500
+Connection ~ 3700 4500
+Wire Wire Line
+	3000 3300 3800 3300
+Wire Wire Line
+	3800 3300 3800 4350
+Connection ~ 3800 4350
+Wire Wire Line
+	3000 3200 3900 3200
+Wire Wire Line
+	3900 3200 3900 4200
+Connection ~ 3900 4200
+Wire Wire Line
+	3000 3900 3200 3900
+Wire Wire Line
+	3000 3100 4100 3100
+Wire Wire Line
+	4100 3100 4100 5600
+Connection ~ 4300 5600
+Wire Wire Line
+	3000 3000 4200 3000
+Wire Wire Line
+	4200 3000 4200 4000
+Wire Wire Line
+	4200 4000 4800 4000
+Connection ~ 4800 4000
+Wire Wire Line
+	5150 3650 4800 3650
+Connection ~ 4800 3650
+$Comp
+L GND #PWR03
+U 1 1 5A32552E
+P 5150 4100
+F 0 "#PWR03" H 5150 3850 50  0001 C CNN
+F 1 "GND" H 5150 3950 50  0000 C CNN
+F 2 "" H 5150 4100 50  0001 C CNN
+F 3 "" H 5150 4100 50  0001 C CNN
+	1    5150 4100
+	1    0    0    -1
+$EndComp
+Wire Wire Line
+	5150 3950 5150 4100
 $EndSCHEMATC
