File: Schematics/ControlBusLEDs/ControlBusLEDs.sch (KiCad schematic (older format))
At the start: 19 parts, among them J1 Conn_01x10, M1 LED_ALT, U2 74HC240

Commit message: Update schematics to KiCad 5
Parts:
- BUSACK1, BUSRQ1, HALT1, IORQ1, M1, MREQ1, RD1, WR1: symbol LED_ALT -> Device:LED_ALT
- C1: symbol C -> Device:C
- J1: symbol Conn_01x10 -> conn:Conn_01x10
- R1, R2, R3, R4, R5, R6, R7, R8: symbol R -> Device:R
- U2: symbol 74HC240 -> ControlBusLEDs-rescue:74HC240
Connections:
- wire segments 98 -> 119
Changed lines of the file:
@@
-EESchema Schematic File Version 2
-LIBS:power
-LIBS:device
-LIBS:switches
-LIBS:relays
-LIBS:motors
-LIBS:transistors
-LIBS:conn
-LIBS:linear
-LIBS:regul
-LIBS:74xx
-LIBS:cmos4000
-LIBS:adc-dac
-LIBS:memory
-LIBS:xilinx
-LIBS:microcontrollers
-LIBS:dsp
-LIBS:microchip
-LIBS:analog_switches
-LIBS:motorola
-LIBS:texas
-LIBS:intel
-LIBS:audio
-LIBS:interface
-LIBS:digital-audio
-LIBS:philips
-LIBS:display
-LIBS:cypress
-LIBS:siliconi
-LIBS:opto
-LIBS:atmel
-LIBS:contrib
-LIBS:valves
-LIBS:Zilog
+EESchema Schematic File Version 4
 LIBS:ControlBusLEDs-cache
-EELAYER 25 0
+EELAYER 26 0
 EELAYER END
 $Descr A4 11693 8268
@@
 $EndDescr
 $Comp
-L 74HC240 U2
+L ControlBusLEDs-rescue:74HC240 U2
 U 1 1 5A1D0470
 P 4800 4800
@@
 $EndComp
 $Comp
-L R R8
+L Device:R R8
 U 1 1 5A1D062F
 P 5800 5000
@@
 $EndComp
 $Comp
-L R R7
+L Device:R R7
 U 1 1 5A1D06E3
 P 5800 4850
@@
 $EndComp
 $Comp
-L R R6
+L Device:R R6
 U 1 1 5A1D06F4
 P 5800 4700
@@
 $EndComp
 $Comp
-L R R5
+L Device:R R5
 U 1 1 5A1D0705
 P 5800 4550
@@
 $EndComp
 $Comp
-L R R4
+L Device:R R4
 U 1 1 5A1D0718
 P 5800 4400
@@
 $EndComp
 $Comp
-L R R3
+L Device:R R3
 U 1 1 5A1D0729
 P 5800 4250
@@
 $EndComp
 $Comp
-L R R2
+L Device:R R2
 U 1 1 5A1D073A
 P 5800 4100
@@
 $EndComp
 $Comp
-L R R1
+L Device:R R1
 U 1 1 5A1D074B
 P 5800 3950
@@
 $EndComp
 $Comp
-L LED_ALT M1
+L Device:LED_ALT M1
 U 1 1 5A1D07CB
 P 7200 5000
@@
 $EndComp
 $Comp
-L LED_ALT HALT1
+L Device:LED_ALT HALT1
 U 1 1 5A1D08CA
 P 7200 4750
@@
 $EndComp
 $Comp
-L LED_ALT RD1
+L Device:LED_ALT RD1
 U 1 1 5A1D08F0
 P 7200 4500
@@
 $EndComp
 $Comp
-L LED_ALT WR1
+L Device:LED_ALT WR1
 U 1 1 5A1D091B
 P 7200 4250
@@
 $EndComp
 $Comp
-L LED_ALT MREQ1
+L Device:LED_ALT MREQ1
 U 1 1 5A1D0947
 P 7200 4000
@@
 $EndComp
 $Comp
-L LED_ALT IORQ1
+L Device:LED_ALT IORQ1
 U 1 1 5A1D0976
 P 7200 3750
@@
 $EndComp
 $Comp
-L LED_ALT BUSRQ1
+L Device:LED_ALT BUSRQ1
 U 1 1 5A1D09A8
 P 7200 3500
@@
 $EndComp
 $Comp
-L LED_ALT BUSACK1
+L Device:LED_ALT BUSACK1
 U 1 1 5A1D0B11
 P 7200 3250
@@
 $EndComp
 $Comp
-L VCC #PWR01
+L power:VCC #PWR01
 U 1 1 5A2D11F3
 P 4800 3550
@@
 $EndComp
 $Comp
-L GND #PWR02
+L power:GND #PWR02
 U 1 1 5A2D128B
 P 4800 5800
@@
 1.01
 $Comp
-L Conn_01x10 J1
+L conn:Conn_01x10 J1
 U 1 1 5A324482
 P 2800 3500
@@
 $EndComp
 $Comp
-L C C1
+L Device:C C1
 U 1 1 5A32538A
 P 5150 3800
@@
 Connection ~ 7750 5000
 Wire Wire Line
-	4800 3550 4800 4100
-Wire Wire Line
-	7750 3250 7750 5600
-Wire Wire Line
-	7750 5600 4100 5600
-Wire Wire Line
-	4800 5500 4800 5800
+	4800 3550 4800 3650
+Wire Wire Line
+	7750 3250 7750 3500
+Wire Wire Line
+	7750 5600 4800 5600
+Wire Wire Line
+	4800 5500 4800 5600
 Connection ~ 4800 5600
 Wire Wire Line
-	4300 5600 4300 5200
+	4300 5600 4300 5300
 Connection ~ 4300 5300
 Wire Wire Line
-	3150 4200 4000 4200
+	3150 4200 3900 4200
 Wire Wire Line
 	4000 4200 4000 4300
@@
 	4000 4300 4300 4300
 Wire Wire Line
-	3150 4350 3900 4350
+	3150 4350 3800 4350
 Wire Wire Line
 	3900 4350 3900 4400
@@
 	3900 4400 4300 4400
 Wire Wire Line
-	3150 4500 4300 4500
-Wire Wire Line
-	3150 4650 3900 4650
+	3150 4500 3700 4500
+Wire Wire Line
+	3150 4650 3600 4650
 Wire Wire Line
 	3900 4650 3900 4600
@@
 	3900 4600 4300 4600
 Wire Wire Line
-	3150 4800 3900 4800
+	3150 4800 3500 4800
 Wire Wire Line
 	3900 4800 3900 4700
@@
 	3900 4700 4300 4700
 Wire Wire Line
-	3150 4950 4000 4950
+	3150 4950 3400 4950
 Wire Wire Line
 	4000 4950 4000 4800
@@
 	4000 4800 4300 4800
 Wire Wire Line
-	3150 5100 4050 5100
+	3150 5100 3300 5100
 Wire Wire Line
 	4050 5100 4050 4900
@@
 	4050 4900 4300 4900
 Wire Wire Line
-	3150 5250 4150 5250
+	3150 5250 3200 5250
 Wire Wire Line
 	4150 5250 4150 5000
@@
 Connection ~ 4800 3650
 $Comp
-L GND #PWR03
+L power:GND #PWR03
 U 1 1 5A32552E
 P 5150 4100
@@
 Wire Wire Line
 	5150 3950 5150 4100
+Wire Wire Line
+	7750 3500 7750 3750
+Wire Wire Line
+	7750 3750 7750 4000
+Wire Wire Line
+	7750 4000 7750 4250
+Wire Wire Line
+	7750 4250 7750 4500
+Wire Wire Line
+	7750 4500 7750 4750
+Wire Wire Line
+	7750 4750 7750 5000
+Wire Wire Line
+	7750 5000 7750 5600
+Wire Wire Line
+	4800 5600 4300 5600
+Wire Wire Line
+	4800 5600 4800 5800
+Wire Wire Line
+	4300 5300 4300 5200
+Wire Wire Line
+	3200 5250 4150 5250
+Wire Wire Line
+	3300 5100 4050 5100
+Wire Wire Line
+	3400 4950 4000 4950
+Wire Wire Line
+	3500 4800 3900 4800
+Wire Wire Line
+	3600 4650 3900 4650
+Wire Wire Line
+	3700 4500 4300 4500
+Wire Wire Line
+	3800 4350 3900 4350
+Wire Wire Line
+	3900 4200 4000 4200
+Wire Wire Line
+	4300 5600 4100 5600
+Wire Wire Line
+	4800 4000 4800 4100
+Wire Wire Line
+	4800 3650 4800 4000
 $EndSCHEMATC

Commit message: Save all Schematics again to overcome problems with version change
Parts:
- J1: symbol conn:Conn_01x10 -> ControlBusLEDs-rescue:Conn_01x10-conn
Changed lines of the file:
@@
 1.01
 $Comp
-L conn:Conn_01x10 J1
+L ControlBusLEDs-rescue:Conn_01x10-conn J1
 U 1 1 5A324482
 P 2800 3500
