File: Schematics/Data bus Spy/DataBusSpy.sch (KiCad schematic (older format))
At the start: 18 parts, among them U1 74HC00, U2 74HCT244

Commit message: Slight changes in DataBus Spy
Parts:
- gave numbers to parts that had none: 7
Connections:
- net labels added: ~RD, ~WR
- net labels removed: RD, WR
Other:
- note added: "1.01"
- note removed: "1.0"
Changed lines of the file:
@@
 10/12/17
 Text Notes 10600 7650 0    60   ~ 0
-1.0
+1.01
 $Comp
 L 74HCT244 U2
@@
 U 1 1 5A1C9B0D
 P 8400 3050
-F 0 "D0" H 8400 3150 50  0001 C CNN
+F 0 "D0" H 8400 3150 50  0000 C CNN
 F 1 "LED" H 8400 2950 50  0001 C CNN
 F 2 "" H 8400 3050 50  0001 C CNN
@@
 $EndComp
 $Comp
-L LED D?
+L LED D1
 U 1 1 5A1C9B6F
 P 8400 3250
-F 0 "D?" H 8400 3350 50  0001 C CNN
+F 0 "D1" H 8400 3350 50  0000 C CNN
 F 1 "LED" H 8400 3150 50  0001 C CNN
 F 2 "" H 8400 3250 50  0001 C CNN
@@
 $EndComp
 $Comp
-L LED D?
+L LED D2
 U 1 1 5A1C9B8C
 P 8400 3450
-F 0 "D?" H 8400 3550 50  0001 C CNN
+F 0 "D2" H 8400 3550 50  0000 C CNN
 F 1 "LED" H 8400 3350 50  0001 C CNN
 F 2 "" H 8400 3450 50  0001 C CNN
@@
 $EndComp
 $Comp
-L LED D?
+L LED D3
 U 1 1 5A1C9BA9
 P 8400 3650
-F 0 "D?" H 8400 3750 50  0001 C CNN
+F 0 "D3" H 8400 3750 50  0000 C CNN
 F 1 "LED" H 8400 3550 50  0001 C CNN
 F 2 "" H 8400 3650 50  0001 C CNN
@@
 $EndComp
 $Comp
-L LED D?
+L LED D4
 U 1 1 5A1C9BC6
 P 8400 3850
-F 0 "D?" H 8400 3950 50  0001 C CNN
+F 0 "D4" H 8400 3950 50  0000 C CNN
 F 1 "LED" H 8400 3750 50  0001 C CNN
 F 2 "" H 8400 3850 50  0001 C CNN
@@
 $EndComp
 $Comp
-L LED D?
+L LED D5
 U 1 1 5A1C9BE3
 P 8400 4050
-F 0 "D?" H 8400 4150 50  0001 C CNN
+F 0 "D5" H 8400 4150 50  0000 C CNN
 F 1 "LED" H 8400 3950 50  0001 C CNN
 F 2 "" H 8400 4050 50  0001 C CNN
@@
 $EndComp
 $Comp
-L LED D?
+L LED D6
 U 1 1 5A1C9C00
 P 8400 4250
-F 0 "D?" H 8400 4350 50  0001 C CNN
+F 0 "D6" H 8400 4350 50  0000 C CNN
 F 1 "LED" H 8400 4150 50  0001 C CNN
 F 2 "" H 8400 4250 50  0001 C CNN
@@
 $EndComp
 $Comp
-L LED D?
+L LED D7
 U 1 1 5A1C9C1D
 P 8400 4450
-F 0 "D?" H 8400 4550 50  0001 C CNN
+F 0 "D7" H 8400 4550 50  0000 C CNN
 F 1 "LED" H 8400 4350 50  0001 C CNN
 F 2 "" H 8400 4450 50  0001 C CNN
@@
 	6850 2850 6850 2700
 Text GLabel 2550 3900 0    60   Input ~ 0
-RD
+~RD
 Text GLabel 2550 4100 0    60   Input ~ 0
-WR
+~WR
 Wire Wire Line
 	2750 3900 2550 3900

Commit message: Add Data Bus Spy PCB and custom footprint library
Parts:
- added 100nf1: C1, Capacitors_THT:C_Disc_D10.0mm_W2.5mm_P5.00mm, symbol C
- added C2: 100 nf, Capacitors_THT:C_Disc_D10.0mm_W2.5mm_P5.00mm, symbol C
- added J1: Conn_01x12, RainbowLibrary:Pin_Header_Straight_1x12_thickpad, symbol Conn_01x12
- D0, D1, D2, D3, D4, D5, D6, D7: footprint (none) -> RainbowLibrary:LED_thickpad
- R1, R2, R3, R4, R5, R6, R7, R8: renamed from R?; footprint (none) -> RainbowLibrary:Resistor_thickpad
- U1: footprint (none) -> RainbowLibrary:DIP-14_thickpad
- U2: footprint (none) -> RainbowLibrary:DIP-20_thickpad
Connections:
- wire segments 81 -> 112
Other:
- moved on the sheet: U1A, U1B, U2

Commit message: Update schematics to KiCad 5
Parts:
- 100nf1, C2: symbol C -> Device:C
- D0, D1, D2, D3, D4, D5, D6, D7: symbol LED -> Device:LED
- J1: symbol Conn_01x12 -> conn:Conn_01x12
- R1, R2, R3, R4, R5, R6, R7, R8: symbol R -> Device:R
- U1: symbol 74HC00 -> DataBusSpy-rescue:74HC00
- U2: symbol 74HCT244 -> DataBusSpy-rescue:74HCT244
Connections:
- wire segments 112 -> 141
Changed lines of the file:
@@
-EESchema Schematic File Version 2
-LIBS:Zilog
-LIBS:power
-LIBS:device
-LIBS:switches
-LIBS:relays
-LIBS:motors
-LIBS:transistors
-LIBS:conn
-LIBS:linear
-LIBS:regul
-LIBS:74xx
-LIBS:cmos4000
-LIBS:adc-dac
-LIBS:memory
-LIBS:xilinx
-LIBS:microcontrollers
-LIBS:dsp
-LIBS:microchip
-LIBS:analog_switches
-LIBS:motorola
-LIBS:texas
-LIBS:intel
-LIBS:audio
-LIBS:interface
-LIBS:digital-audio
-LIBS:philips
-LIBS:display
-LIBS:cypress
-LIBS:siliconi
-LIBS:opto
-LIBS:atmel
-LIBS:contrib
-LIBS:valves
-LIBS:cmos_ieee
+EESchema Schematic File Version 4
 LIBS:DataBusSpy-cache
-EELAYER 25 0
+EELAYER 26 0
 EELAYER END
 $Descr A4 11693 8268
@@
 1.01
 $Comp
-L 74HCT244 U2
+L DataBusSpy-rescue:74HCT244 U2
 U 1 1 5A1C8654
 P 6100 3550
@@
 $EndComp
 $Comp
-L R R1
+L Device:R R1
 U 1 1 5A1C93CE
 P 7200 3050
@@
 $EndComp
 $Comp
-L R R2
+L Device:R R2
 U 1 1 5A1C943E
 P 7200 3250
@@
 $EndComp
 $Comp
-L R R3
+L Device:R R3
 U 1 1 5A1C946E
 P 7200 3450
@@
 $EndComp
 $Comp
-L R R4
+L Device:R R4
 U 1 1 5A1C949D
 P 7200 3650
@@
 $EndComp
 $Comp
-L R R5
+L Device:R R5
 U 1 1 5A1C94DD
 P 7200 3850
@@
 $EndComp
 $Comp
-L R R6
+L Device:R R6
 U 1 1 5A1C95D7
 P 7200 4050
@@
 $EndComp
 $Comp
-L R R7
+L Device:R R7
 U 1 1 5A1C960F
 P 7200 4250
@@
 $EndComp
 $Comp
-L R R8
+L Device:R R8
 U 1 1 5A1C9652
 P 7200 4450
@@
 $EndComp
 $Comp
-L LED D0
+L Device:LED D0
 U 1 1 5A1C9B0D
 P 7650 3050
@@
 $EndComp
 $Comp
-L LED D1
+L Device:LED D1
 U 1 1 5A1C9B6F
 P 7650 3250
@@
 $EndComp
 $Comp
-L LED D2
+L Device:LED D2
 U 1 1 5A1C9B8C
 P 7650 3450
@@
 $EndComp
 $Comp
-L LED D3
+L Device:LED D3
 U 1 1 5A1C9BA9
 P 7650 3650
@@
 $EndComp
 $Comp
-L LED D4
+L Device:LED D4
 U 1 1 5A1C9BC6
 P 7650 3850
@@
 $EndComp
 $Comp
-L LED D5
+L Device:LED D5
 U 1 1 5A1C9BE3
 P 7650 4050
@@
 $EndComp
 $Comp
-L LED D6
+L Device:LED D6
 U 1 1 5A1C9C00
 P 7650 4250
@@
 $EndComp
 $Comp
-L LED D7
+L Device:LED D7
 U 1 1 5A1C9C1D
 P 7650 4450
@@
 $EndComp
 $Comp
-L 74HC00 U1
+L DataBusSpy-rescue:74HC00 U1
 U 1 1 5A2D332F
 P 3950 5050
@@
 $EndComp
 $Comp
-L 74HC00 U1
+L DataBusSpy-rescue:74HC00 U1
 U 2 1 5A2D35C9
 P 5200 5050
@@
 $EndComp
 $Comp
-L GND #PWR2
+L power:GND #PWR2
 U 1 1 5A2D3813
 P 6100 4850
@@
 $EndComp
 $Comp
-L VCC #PWR1
+L power:VCC #PWR1
 U 1 1 5A2D386A
 P 6100 1850
@@
 Connection ~ 8000 4450
 Wire Wire Line
-	8000 3050 8000 4700
+	8000 3050 8000 3250
 Wire Wire Line
 	5600 3950 5450 3950
 Wire Wire Line
-	5450 3950 5450 4050
+	5450 3950 5450 4000
 Wire Wire Line
 	5450 4050 5600 4050
 Wire Wire Line
-	4600 4950 4600 5150
+	4600 4950 4600 5050
 Wire Wire Line
 	4550 5050 4600 5050
@@
 Connection ~ 5450 4000
 Wire Wire Line
-	6100 4250 6100 4850
+	6100 4250 6100 4700
 Connection ~ 6100 4700
 Wire Wire Line
-	6100 1850 6100 2850
-Wire Wire Line
-	3350 4950 3150 4950
-Wire Wire Line
-	3350 5150 3150 5150
-Wire Wire Line
-	4400 2800 5600 2800
-Wire Wire Line
-	4400 2950 5550 2950
-Wire Wire Line
-	4400 3400 5550 3400
-Wire Wire Line
-	4400 3550 5600 3550
-Wire Wire Line
-	4400 3700 5450 3700
+	6100 1850 6100 1950
+Wire Wire Line
+	3350 4950 3250 4950
+Wire Wire Line
+	3350 5150 3300 5150
+Wire Wire Line
+	4400 2800 5300 2800
+Wire Wire Line
+	4400 2950 5200 2950
+Wire Wire Line
+	4400 3400 4900 3400
+Wire Wire Line
+	4400 3550 4800 3550
+Wire Wire Line
+	4400 3700 4700 3700
 Wire Wire Line
 	5450 3700 5450 3650
@@
 	5450 3650 5600 3650
 Wire Wire Line
-	4400 3850 5500 3850
+	4400 3850 4600 3850
 Wire Wire Line
 	5500 3850 5500 3750
@@
 	5550 3450 5600 3450
 Wire Wire Line
-	4400 3250 5400 3250
+	4400 3250 5000 3250
 Wire Wire Line
 	5400 3250 5400 3350
@@
 	5400 3350 5600 3350
 Wire Wire Line
-	4400 3100 5450 3100
+	4400 3100 5100 3100
 Wire Wire Line
 	5450 3100 5450 3250
@@
 	5000 5250 5000 5450
 Wire Wire Line
-	3750 5450 8550 5450
+	3750 5450 5000 5450
 Wire Wire Line
 	3750 5450 3750 5250
@@
 	5000 4850 5000 4600
 Wire Wire Line
-	3750 4600 8400 4600
-Connection ~ 3750 4850
+	3750 4600 5000 4600
 Wire Wire Line
 	3750 4600 3750 4850
@@
 	8400 4600 8400 2650
 Wire Wire Line
-	8400 2650 5900 2650
+	8400 2650 6100 2650
 Connection ~ 6100 2650
 Connection ~ 5000 4600
@@
 Connection ~ 5300 2800
 Wire Wire Line
-	8000 4700 6100 4700
-$Comp
-L Conn_01x12 J1
+	8000 4700 6550 4700
+$Comp
+L conn:Conn_01x12 J1
 U 1 1 5A32DECF
 P 2850 2350
@@
 Connection ~ 3300 5150
 $Comp
-L C C2
+L Device:C C2
 U 1 1 5A339617
 P 6450 2100
@@
 $EndComp
 $Comp
-L C 100nf1
+L Device:C 100nf1
 U 1 1 5A3399E1
 P 8250 4850
@@
 Connection ~ 6100 1950
 $Comp
-L GND #PWR3
+L power:GND #PWR3
 U 1 1 5A33A746
 P 6450 2350
@@
 Wire Wire Line
 	6450 2250 6450 2350
+Wire Wire Line
+	8000 3250 8000 3450
+Wire Wire Line
+	8000 3450 8000 3650
+Wire Wire Line
+	8000 3650 8000 3850
+Wire Wire Line
+	8000 3850 8000 4050
+Wire Wire Line
+	8000 4050 8000 4250
+Wire Wire Line
+	8000 4250 8000 4450
+Wire Wire Line
+	8000 4450 8000 4700
+Wire Wire Line
+	4600 5050 4600 5150
+Wire Wire Line
+	5450 4000 5450 4050
+Wire Wire Line
+	6100 4700 6100 4850
+Wire Wire Line
+	5000 5450 6550 5450
+Wire Wire Line
+	6550 4700 6100 4700
+Wire Wire Line
+	6100 2650 6100 2850
+Wire Wire Line
+	6100 2650 5900 2650
+Wire Wire Line
+	5000 4600 8250 4600
+Wire Wire Line
+	6550 5450 8250 5450
+Wire Wire Line
+	4600 3850 5500 3850
+Wire Wire Line
+	4700 3700 5450 3700
+Wire Wire Line
+	4800 3550 5600 3550
+Wire Wire Line
+	4900 3400 5550 3400
+Wire Wire Line
+	5000 3250 5400 3250
+Wire Wire Line
+	5100 3100 5450 3100
+Wire Wire Line
+	5200 2950 5550 2950
+Wire Wire Line
+	5300 2800 5600 2800
+Wire Wire Line
+	3250 4950 3150 4950
+Wire Wire Line
+	3300 5150 3150 5150
+Wire Wire Line
+	8250 4600 8400 4600
+Wire Wire Line
+	8250 5450 8550 5450
+Wire Wire Line
+	6100 1950 6100 2650
 $EndSCHEMATC

Commit message: Save all Schematics again to overcome problems with version change
Parts:
- J1: symbol conn:Conn_01x12 -> DataBusSpy-rescue:Conn_01x12-conn
Changed lines of the file:
@@
 	8000 4700 6550 4700
 $Comp
-L conn:Conn_01x12 J1
+L DataBusSpy-rescue:Conn_01x12-conn J1
 U 1 1 5A32DECF
 P 2850 2350
