File: Schematics/Intelligent Display Interface/idi.sch (KiCad schematic (older format))
At the start: 25 parts, among them U1 MSP430G2553_PW20, U2 74HC244

Commit message: Add a buffer stage for the IORQ signal in IDI - required for reliable operation
Parts:
- added U1: 74HC04, symbol 74HC04
- added unit 2 of U1
Connections:
- wire segments 116 -> 127
Other:
- moved on the sheet: RV1, U2

Commit message: Update schematics to KiCad 5
Parts:
- C1: symbol C_Small -> Device:C_Small
- DS1: symbol HY1602E -> display:HY1602E
- R1, R10, R11, R12, R13, R14, R15, R16, R17, R18, R19, R2, R3, R4, R5, R6, R7, R8, R9: symbol R -> Device:R
- RV1: symbol POT_TRIM -> idi-rescue:POT_TRIM
- U1: symbol MSP430G2553_PW20 -> mymsp430:MSP430G2553_PW20
- U1: symbol 74HC04 -> idi-rescue:74HC04
- U2: symbol 74HC244 -> idi-rescue:74HC244
Connections:
- wire segments 127 -> 163
Changed lines of the file:
@@
-EESchema Schematic File Version 2
-LIBS:power
-LIBS:device
-LIBS:switches
-LIBS:relays
-LIBS:motors
-LIBS:transistors
-LIBS:conn
-LIBS:linear
-LIBS:regul
-LIBS:74xx
-LIBS:cmos4000
-LIBS:adc-dac
-LIBS:memory
-LIBS:xilinx
-LIBS:microcontrollers
-LIBS:dsp
-LIBS:microchip
-LIBS:analog_switches
-LIBS:motorola
-LIBS:texas
-LIBS:intel
-LIBS:audio
-LIBS:interface
-LIBS:digital-audio
-LIBS:philips
-LIBS:display
-LIBS:cypress
-LIBS:siliconi
-LIBS:opto
-LIBS:atmel
-LIBS:contrib
-LIBS:valves
-LIBS:mymsp430
+EESchema Schematic File Version 4
 LIBS:idi-cache
-EELAYER 25 0
+EELAYER 26 0
 EELAYER END
 $Descr A4 11693 8268
@@
 $EndDescr
 $Comp
-L MSP430G2553_PW20 U1
+L mymsp430:MSP430G2553_PW20 U1
 U 1 1 5A5C57F3
 P 6800 3400
@@
 $EndComp
 $Comp
-L HY1602E DS1
+L display:HY1602E DS1
 U 1 1 5A5C5933
 P 9400 3450
@@
 $EndComp
 $Comp
-L +3.3V #PWR1
+L power:+3.3V #PWR1
 U 1 1 5A5C5BC4
 P 5800 3750
@@
 $EndComp
 $Comp
-L +5V #PWR2
+L power:+5V #PWR2
 U 1 1 5A5C62D9
 P 9400 2400
@@
 $EndComp
 $Comp
-L GND #PWR3
+L power:GND #PWR3
 U 1 1 5A5C64B4
 P 9400 4400
@@
 $EndComp
 $Comp
-L POT_TRIM RV1
+L idi-rescue:POT_TRIM RV1
 U 1 1 5A5C67CF
 P 10500 2850
@@
 $EndComp
 $Comp
-L 74HC244 U2
+L idi-rescue:74HC244 U2
 U 1 1 5A5C7805
 P 2800 3350
@@
 $EndComp
 $Comp
-L R R2
+L Device:R R2
 U 1 1 5A5C81CA
 P 4350 3900
@@
 $EndComp
 $Comp
-L R R3
+L Device:R R3
 U 1 1 5A5C8214
 P 4550 3900
@@
 $EndComp
 $Comp
-L R R4
+L Device:R R4
 U 1 1 5A5C823E
 P 4750 3900
@@
 $EndComp
 $Comp
-L R R5
+L Device:R R5
 U 1 1 5A5C8276
 P 4950 3900
@@
 $EndComp
 $Comp
-L R R6
+L Device:R R6
 U 1 1 5A5C82B2
 P 5150 3900
@@
 $EndComp
 $Comp
-L R R7
+L Device:R R7
 U 1 1 5A5C82E5
 P 5350 3900
@@
 $EndComp
 $Comp
-L R R8
+L Device:R R8
 U 1 1 5A5C8317
 P 5550 3900
@@
 $EndComp
 $Comp
-L R R1
+L Device:R R1
 U 1 1 5A5C8354
 P 4150 3900
@@
 $EndComp
 $Comp
-L R R9
+L Device:R R9
 U 1 1 5A5C87A2
 P 5050 2850
@@
 $EndComp
 $Comp
-L R R10
+L Device:R R10
 U 1 1 5A5C8A1A
 P 4900 2950
@@
 $EndComp
 $Comp
-L R R11
+L Device:R R11
 U 1 1 5A5C8BEB
 P 4700 3050
@@
 $EndComp
 $Comp
-L R R12
+L Device:R R12
 U 1 1 5A5C8E25
 P 4500 3150
@@
 $EndComp
 $Comp
-L R R13
+L Device:R R13
 U 1 1 5A5C8F89
 P 4300 3250
@@
 $EndComp
 $Comp
-L R R14
+L Device:R R14
 U 1 1 5A5C91C0
 P 4100 3350
@@
 $EndComp
 $Comp
-L R R15
+L Device:R R15
 U 1 1 5A5C9381
 P 3900 3450
@@
 $EndComp
 $Comp
-L R R16
+L Device:R R16
 U 1 1 5A5C959F
 P 3700 3550
@@
 ~IORQ
 $Comp
-L R R17
+L Device:R R17
 U 1 1 5A5CCF23
 P 3700 4500
@@
 $EndComp
 $Comp
-L R R18
+L Device:R R18
 U 1 1 5A5CD05B
 P 3700 4950
@@
 1.0a
 $Comp
-L R R19
+L Device:R R19
 U 1 1 5A5CF61B
 P 8300 4950
@@
 $EndComp
 $Comp
-L C_Small C1
+L Device:C_Small C1
 U 1 1 5A5CF7DC
 P 8300 4550
@@
 JTAG_SWBCLK
 $Comp
-L R R19
+L Device:R R19
 U 1 1 5A5D23FF
 P 8750 4900
@@
 	8900 2850 9000 2850
 Wire Wire Line
-	9400 2400 9400 2650
-Wire Wire Line
-	9400 4250 9400 4400
+	9400 2400 9400 2500
+Wire Wire Line
+	9400 4250 9400 4300
 Wire Wire Line
 	9800 3450 10000 3450
@@
 	10000 3450 10000 2500
 Wire Wire Line
-	1050 2500 10500 2500
+	1050 2500 2800 2500
 Connection ~ 9400 2500
 Wire Wire Line
@@
 	8600 3050 8600 4300
 Wire Wire Line
-	5800 3750 5950 3750
+	5800 3750 5900 3750
 Wire Wire Line
 	5950 4050 5700 4050
@@
 	5550 4300 5550 4050
 Wire Wire Line
-	5200 2850 5950 2850
-Wire Wire Line
-	5050 2950 5950 2950
-Wire Wire Line
-	4850 3050 5950 3050
-Wire Wire Line
-	4650 3150 5950 3150
-Wire Wire Line
-	4450 3250 5950 3250
-Wire Wire Line
-	4250 3350 5950 3350
-Wire Wire Line
-	4050 3450 5950 3450
-Wire Wire Line
-	3850 3550 5950 3550
-Wire Wire Line
-	2800 4300 10500 4300
+	5200 2850 5550 2850
+Wire Wire Line
+	5050 2950 5350 2950
+Wire Wire Line
+	4850 3050 5150 3050
+Wire Wire Line
+	4650 3150 4950 3150
+Wire Wire Line
+	4450 3250 4750 3250
+Wire Wire Line
+	4250 3350 4550 3350
+Wire Wire Line
+	4050 3450 4350 3450
+Wire Wire Line
+	3850 3550 4150 3550
+Wire Wire Line
+	2800 4300 3700 4300
 Connection ~ 5550 4300
 Connection ~ 5350 4300
@@
 	2250 3850 2300 3850
 Wire Wire Line
-	2250 4050 1600 4050
+	2250 4050 1700 4050
 Connection ~ 2250 3850
 Wire Wire Line
@@
 	8300 4450 8300 4300
 Wire Wire Line
-	8300 4650 8300 4800
+	8300 4650 8300 4700
 Wire Wire Line
 	8300 5100 8300 5250
@@
 Connection ~ 5900 3750
 Wire Wire Line
-	8150 4700 9000 4700
+	8150 4700 8300 4700
 Connection ~ 8300 4700
 Wire Wire Line
@@
 	8150 4950 8150 4700
 $Comp
-L 74HC04 U1
+L idi-rescue:74HC04 U1
 U 1 1 5AA24377
 P 2150 5100
@@
 $EndComp
 $Comp
-L 74HC04 U1
+L idi-rescue:74HC04 U1
 U 2 1 5AA24527
 P 2950 5100
@@
 	2800 4050 2800 4300
 Wire Wire Line
-	3700 4650 3700 4800
+	3700 4650 3700 4750
 Connection ~ 3700 4750
 Wire Wire Line
@@
 	3400 5100 3700 5100
 Wire Wire Line
-	2250 3750 2250 4050
+	2250 3750 2250 3850
 Wire Wire Line
 	1700 5100 1700 4050
@@
 	2900 4750 2900 5000
 Wire Wire Line
-	1050 4750 2900 4750
+	1050 4750 2100 4750
 Wire Wire Line
 	2100 4750 2100 5000
@@
 	2900 5200 2900 5400
 Wire Wire Line
-	2100 5400 4000 5400
+	2100 5400 2900 5400
 Wire Wire Line
 	2100 5400 2100 5200
@@
 Connection ~ 4000 4300
 Connection ~ 2900 5400
+Wire Wire Line
+	9400 2500 9400 2650
+Wire Wire Line
+	9400 2500 10000 2500
+Wire Wire Line
+	9400 4300 9400 4400
+Wire Wire Line
+	9400 4300 10000 4300
+Wire Wire Line
+	10000 2500 10500 2500
+Wire Wire Line
+	10000 4300 10500 4300
+Wire Wire Line
+	8600 4300 9400 4300
+Wire Wire Line
+	5700 4300 8300 4300
+Wire Wire Line
+	5550 4300 5700 4300
+Wire Wire Line
+	5350 4300 5550 4300
+Wire Wire Line
+	5150 4300 5350 4300
+Wire Wire Line
+	4950 4300 5150 4300
+Wire Wire Line
+	4750 4300 4950 4300
+Wire Wire Line
+	4550 4300 4750 4300
+Wire Wire Line
+	4350 4300 4550 4300
+Wire Wire Line
+	4150 4300 4350 4300
+Wire Wire Line
+	4150 3550 5950 3550
+Wire Wire Line
+	4350 3450 5950 3450
+Wire Wire Line
+	4550 3350 5950 3350
+Wire Wire Line
+	4750 3250 5950 3250
+Wire Wire Line
+	4950 3150 5950 3150
+Wire Wire Line
+	5150 3050 5950 3050
+Wire Wire Line
+	5350 2950 5950 2950
+Wire Wire Line
+	5550 2850 5950 2850
+Wire Wire Line
+	2250 3850 2250 4050
+Wire Wire Line
+	8300 4300 8600 4300
+Wire Wire Line
+	5900 3750 5950 3750
+Wire Wire Line
+	8300 4700 8300 4800
+Wire Wire Line
+	8300 4700 9000 4700
+Wire Wire Line
+	3700 4750 3700 4800
+Wire Wire Line
+	3700 4300 4000 4300
+Wire Wire Line
+	1700 4050 1600 4050
+Wire Wire Line
+	2800 2500 9400 2500
+Wire Wire Line
+	2100 4750 2900 4750
+Wire Wire Line
+	4000 4300 4150 4300
+Wire Wire Line
+	2900 5400 4000 5400
 $EndSCHEMATC

Commit message: Save all Schematics again to overcome problems with version change
Parts:
- DS1: symbol display:HY1602E -> idi-rescue:HY1602E-display
Changed lines of the file:
@@
 $EndComp
 $Comp
-L display:HY1602E DS1
+L idi-rescue:HY1602E-display DS1
 U 1 1 5A5C5933
 P 9400 3450
