File: Schematics/ProgrammableClock/ProgrammableClock.sch (KiCad schematic (older format))
At the start: 26 parts, among them J1 Board Connection, SW1 Up_freq, SW2 Down_freq, SW3 Multiply, SW4 Step, U1 MSP430G2553_PW20, U2 74HC244

Commit message: Update schematics to KiCad 5
Parts:
- C1, C2, C3, C4, C5, C6, C7: symbol C -> Device:C
- D1: symbol LED -> Device:LED
- J1: symbol Conn_01x05 -> conn:Conn_01x05
- R1, R10, R2, R3, R4, R5, R6, R7, R8, R9: symbol R -> Device:R
- SW1, SW2, SW3, SW4: symbol SW_Push -> switches:SW_Push
- U1: symbol MSP430G2553_PW20 -> mymsp430:MSP430G2553_PW20
- U2: symbol 74HC244 -> ProgrammableClock-rescue:74HC244
Connections:
- wire segments 102 -> 136

Commit message: Save all Schematics again to overcome problems with version change
Parts:
- J1: symbol conn:Conn_01x05 -> ProgrammableClock-rescue:Conn_01x05-conn
- SW1, SW2, SW3, SW4: symbol switches:SW_Push -> ProgrammableClock-rescue:SW_Push-switches
Changed lines of the file:
@@
 $EndComp
 $Comp
-L conn:Conn_01x05 J1
+L ProgrammableClock-rescue:Conn_01x05-conn J1
 U 1 1 5AAF8572
 P 3300 2250
@@
 SBW_CLK
 $Comp
-L switches:SW_Push SW1
+L ProgrammableClock-rescue:SW_Push-switches SW1
 U 1 1 5AAF9A84
 P 5800 4050
@@
 $EndComp
 $Comp
-L switches:SW_Push SW2
+L ProgrammableClock-rescue:SW_Push-switches SW2
 U 1 1 5AAF9AE2
 P 5800 4550
@@
 $EndComp
 $Comp
-L switches:SW_Push SW3
+L ProgrammableClock-rescue:SW_Push-switches SW3
 U 1 1 5AAF9B33
 P 5800 5050
@@
 $EndComp
 $Comp
-L switches:SW_Push SW4
+L ProgrammableClock-rescue:SW_Push-switches SW4
 U 1 1 5AB0AE39
 P 5800 5550
