File: Schematics/RAM Test/RamTest.sch (KiCad schematic (older format))
At the start: 36 parts, among them SW2 SW_DIP_x08, U1 6116

Commit message: Update schematics to KiCad 5
Parts:
- C2: symbol C_Small -> Device:C_Small
- C?: symbol CP -> Device:CP
- D? (x8): symbol LED -> Device:LED
- R1, R? (x21): symbol R -> Device:R
- SW2: symbol SW_DIP_x08 -> switches:SW_DIP_x08
- SW?: symbol SW_DIP_x04 -> switches:SW_DIP_x04
- SW?: symbol SW_DIP_x02 -> switches:SW_DIP_x02
- U1: symbol 6116 -> memory:6116

Commit message: Save all Schematics again to overcome problems with version change
Parts:
- SW2: symbol switches:SW_DIP_x08 -> RamTest-rescue:SW_DIP_x08-switches
- SW?: symbol switches:SW_DIP_x04 -> RamTest-rescue:SW_DIP_x04-switches
- SW?: symbol switches:SW_DIP_x02 -> RamTest-rescue:SW_DIP_x02-switches
- U1: symbol memory:6116 -> RamTest-rescue:6116-memory
Changed lines of the file:
@@
 16/12/17
 $Comp
-L switches:SW_DIP_x08 SW2
+L RamTest-rescue:SW_DIP_x08-switches SW2
 U 1 1 5A343A4F
 P 8900 3600
@@
 $EndComp
 $Comp
-L switches:SW_DIP_x04 SW?
+L RamTest-rescue:SW_DIP_x04-switches SW?
 U 1 1 5A343D88
 P 3300 3600
@@
 $EndComp
 $Comp
-L memory:6116 U1
+L RamTest-rescue:6116-memory U1
 U 1 1 5A344BF5
 P 5750 4200
@@
 $EndComp
 $Comp
-L switches:SW_DIP_x02 SW?
+L RamTest-rescue:SW_DIP_x02-switches SW?
 U 1 1 5A344DDB
 P 4000 3600
