File: Schematics/Z80 Mainboard/Z80Mainboard.sch (KiCad schematic (older format))
At the start: 13 parts, among them J1 Address Bus Connector, J2 Data Bus Connector, J3 Control Bus & Power, U1 Atmel 28C64, U2 74HCT138, U3 6116

Commit message: Add revision 1.1 of Z80 Mainboard
Parts:
- added C6: 100nF, symbol C_Small
- added J?: Data Bus Connector (to Display Interface), symbol Conn_01x09
- J1: value Address Bus Connector -> Address Bus Connector (to Bus Spy)
- J2: value Data Bus Connector -> Data Bus Connector (to Data Spy)
- J3: value Control Bus & Power -> Control Bus, Clock & Power
- gave numbers to parts that had none: 1
Connections:
- net labels added: ~BUSACK, ~BUSRQ, ~HALT, ~IORQ, ~M1, ~MREQ, ~RD, ~WR
- net labels removed: BUSACK, BUSRQ, HALT, IORQ, M1, MREQ, RD, WR
- wire segments 197 -> 210
Other:
- note added: "1.1"
- note added: "15/03/2018"
- note removed: "1.0"
- note removed: "22/01/2018"
- moved on the sheet: C1, C2, C3, C4, C5, J1, J2, J3, R1, U1, U2, U3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

Commit message: Update schematics to KiCad 5
Parts:
- C1: symbol CP -> Device:CP
- C2, C3, C4, C5, C6: symbol C_Small -> Device:C_Small
- J1: symbol Conn_01x16 -> conn:Conn_01x16
- J2: symbol Conn_01x08 -> conn:Conn_01x08
- J3: symbol Conn_01x11 -> conn:Conn_01x11
- J?: symbol Conn_01x09 -> conn:Conn_01x09
- R1: symbol R -> Device:R
- U1: symbol 27C64 -> memory:27C64
- U2: symbol 74LS138 -> Z80Mainboard-rescue:74LS138
- U3: symbol 6116 -> memory:6116
- U4: symbol Z80CPU -> Zilog:Z80CPU

Commit message: Save all Schematics again to overcome problems with version change
Parts:
- J1: symbol conn:Conn_01x16 -> Z80Mainboard-rescue:Conn_01x16-conn
- J2: symbol conn:Conn_01x08 -> Z80Mainboard-rescue:Conn_01x08-conn
- J3: symbol conn:Conn_01x11 -> Z80Mainboard-rescue:Conn_01x11-conn
- J?: symbol conn:Conn_01x09 -> Z80Mainboard-rescue:Conn_01x09-conn
- U1: symbol memory:27C64 -> Z80Mainboard-rescue:27C64-memory
- U3: symbol memory:6116 -> Z80Mainboard-rescue:6116-memory
- U4: symbol Zilog:Z80CPU -> Z80Mainboard-rescue:Z80CPU-Zilog
Changed lines of the file:
@@
 $EndDescr
 $Comp
-L memory:6116 U3
+L Z80Mainboard-rescue:6116-memory U3
 U 1 1 5A2E5CEB
 P 9150 4500
@@
 1.1
 $Comp
-L memory:27C64 U1
+L Z80Mainboard-rescue:27C64-memory U1
 U 1 1 5A2E5C26
 P 9150 2350
@@
 $EndComp
 $Comp
-L Zilog:Z80CPU U4
+L Z80Mainboard-rescue:Z80CPU-Zilog U4
 U 1 1 5A65CBFC
 P 2850 3300
@@
 $EndComp
 $Comp
-L conn:Conn_01x16 J1
+L Z80Mainboard-rescue:Conn_01x16-conn J1
 U 1 1 5A67A1D2
 P 2400 6550
@@
 A15
 $Comp
-L conn:Conn_01x08 J2
+L Z80Mainboard-rescue:Conn_01x08-conn J2
 U 1 1 5A67D9E0
 P 3900 6550
@@
 ~BUSACK
 $Comp
-L conn:Conn_01x11 J3
+L Z80Mainboard-rescue:Conn_01x11-conn J3
 U 1 1 5A68C75C
 P 5250 6550
@@
 	5650 6100 5650 6350
 $Comp
-L conn:Conn_01x09 J?
+L Z80Mainboard-rescue:Conn_01x09-conn J?
 U 1 1 5AAA220A
 P 3900 7250
@@
 	2000 1700 2000 1750
 Wire Bus Line
+	1000 2300 1000 5550
+Wire Bus Line
 	4650 6000 5950 6000
-Wire Bus Line
-	1000 2300 1000 5550
 Wire Bus Line
 	3400 6000 4550 6000
 Wire Bus Line
+	3400 6800 4550 6800
+Wire Bus Line
 	3950 3800 3950 5700
 Wire Bus Line
-	3400 6800 4550 6800
-Wire Bus Line
 	10450 1300 10450 5700
