File: Schematics/Z80 and ROM/Z80Rom.sch (KiCad schematic (older format))
At the start: 22 parts, among them U1 Z80ACPU, U2 AT28C64, U3 74HCT244

Commit message: Update schematics to KiCad 5
Parts:
- C1: symbol CP1 -> Device:CP1
- D? (x8): symbol LED -> Device:LED
- R1, R? (x8): symbol R -> Device:R
- SW?: symbol SW_SPST -> switches:SW_SPST
- U1: symbol Z80CPU -> Zilog:Z80CPU
- U2: symbol 27C64 -> memory:27C64
- U3: symbol 74HCT244 -> Z80Rom-rescue:74HCT244
Connections:
- wire segments 126 -> 156
Changed lines of the file:
@@
-EESchema Schematic File Version 2
-LIBS:Zilog
-LIBS:power
-LIBS:device
-LIBS:switches
-LIBS:relays
-LIBS:motors
-LIBS:transistors
-LIBS:conn
-LIBS:linear
-LIBS:regul
-LIBS:74xx
-LIBS:cmos4000
-LIBS:adc-dac
-LIBS:memory
-LIBS:xilinx
-LIBS:microcontrollers
-LIBS:dsp
-LIBS:microchip
-LIBS:analog_switches
-LIBS:motorola
-LIBS:texas
-LIBS:intel
-LIBS:audio
-LIBS:interface
-LIBS:digital-audio
-LIBS:philips
-LIBS:display
-LIBS:cypress
-LIBS:siliconi
-LIBS:opto
-LIBS:atmel
-LIBS:contrib
-LIBS:valves
-LIBS:cmos_ieee
+EESchema Schematic File Version 4
 LIBS:Z80Rom-cache
-EELAYER 25 0
+EELAYER 26 0
 EELAYER END
 $Descr A4 11693 8268
@@
 $EndDescr
 $Comp
-L Z80CPU U1
+L Zilog:Z80CPU U1
 U 1 1 5A1A6EC8
 P 3750 3800
@@
 $EndComp
 $Comp
-L VCC #PWR?
+L power:VCC #PWR?
 U 1 1 5A1A6F3C
 P 1700 2300
@@
 $EndComp
 $Comp
-L GND #PWR?
+L power:GND #PWR?
 U 1 1 5A1A6F76
 P 1700 5350
@@
 $EndComp
 $Comp
-L CP1 C1
+L Device:CP1 C1
 U 1 1 5A1A6FD7
 P 1700 5000
@@
 $EndComp
 $Comp
-L R R1
+L Device:R R1
 U 1 1 5A1A7360
 P 2650 2600
@@
 $EndComp
 $Comp
-L SW_SPST SW?
+L switches:SW_SPST SW?
 U 1 1 5A1A73BF
 P 2450 2900
@@
 1.0
 $Comp
-L 27C64 U2
+L memory:27C64 U2
 U 1 1 5A1C6F65
 P 6000 3500
@@
 $EndComp
 $Comp
-L 74HCT244 U3
+L Z80Rom-rescue:74HCT244 U3
 U 1 1 5A1C8654
 P 7950 3450
@@
 $EndComp
 $Comp
-L R R?
+L Device:R R?
 U 1 1 5A1C93CE
 P 9050 2950
@@
 $EndComp
 $Comp
-L R R?
+L Device:R R?
 U 1 1 5A1C943E
 P 9050 3150
@@
 $EndComp
 $Comp
-L R R?
+L Device:R R?
 U 1 1 5A1C946E
 P 9050 3350
@@
 $EndComp
 $Comp
-L R R?
+L Device:R R?
 U 1 1 5A1C949D
 P 9050 3550
@@
 $EndComp
 $Comp
-L R R?
+L Device:R R?
 U 1 1 5A1C94DD
 P 9050 3750
@@
 $EndComp
 $Comp
-L R R?
+L Device:R R?
 U 1 1 5A1C95D7
 P 9050 3950
@@
 $EndComp
 $Comp
-L R R?
+L Device:R R?
 U 1 1 5A1C960F
 P 9050 4150
@@
 $EndComp
 $Comp
-L R R?
+L Device:R R?
 U 1 1 5A1C9652
 P 9050 4350
@@
 $EndComp
 $Comp
-L LED D?
+L Device:LED D?
 U 1 1 5A1C9B0D
 P 9500 2950
@@
 $EndComp
 $Comp
-L LED D?
+L Device:LED D?
 U 1 1 5A1C9B6F
 P 9500 3150
@@
 $EndComp
 $Comp
-L LED D?
+L Device:LED D?
 U 1 1 5A1C9B8C
 P 9500 3350
@@
 $EndComp
 $Comp
-L LED D?
+L Device:LED D?
 U 1 1 5A1C9BA9
 P 9500 3550
@@
 $EndComp
 $Comp
-L LED D?
+L Device:LED D?
 U 1 1 5A1C9BC6
 P 9500 3750
@@
 $EndComp
 $Comp
-L LED D?
+L Device:LED D?
 U 1 1 5A1C9BE3
 P 9500 3950
@@
 $EndComp
 $Comp
-L LED D?
+L Device:LED D?
 U 1 1 5A1C9C00
 P 9500 4150
@@
 $EndComp
 $Comp
-L LED D?
+L Device:LED D?
 U 1 1 5A1C9C1D
 P 9500 4350
@@
 Connection ~ 1700 2300
 Wire Wire Line
-	9850 5300 1700 5300
-Wire Wire Line
-	1700 5150 1700 5350
+	9850 5300 7950 5300
+Wire Wire Line
+	1700 5150 1700 5300
 Connection ~ 1700 5300
 Wire Wire Line
-	1700 2300 7950 2300
-Wire Wire Line
-	1700 4850 1700 2300
+	1700 2300 2650 2300
+Wire Wire Line
+	1700 4850 1700 4000
 Wire Wire Line
 	3050 3300 1700 3300
@@
 	4450 3800 5300 3800
 Wire Wire Line
-	6700 3300 6700 5000
+	6700 3300 6700 3650
 Wire Wire Line
 	6700 5000 4450 5000
@@
 	6700 3200 6750 3200
 Wire Wire Line
-	6750 3200 6750 4900
+	6750 3200 6750 3550
 Wire Wire Line
 	6750 4900 4450 4900
@@
 	6700 3100 6800 3100
 Wire Wire Line
-	6800 3100 6800 4800
+	6800 3100 6800 3450
 Wire Wire Line
 	6800 4800 4450 4800
@@
 	6700 3000 6850 3000
 Wire Wire Line
-	6850 3000 6850 4700
+	6850 3000 6850 3350
 Wire Wire Line
 	6850 4700 4450 4700
@@
 	6700 2900 6900 2900
 Wire Wire Line
-	6900 2900 6900 4600
+	6900 2900 6900 3250
 Wire Wire Line
 	6900 4600 4450 4600
@@
 	6700 2800 7000 2800
 Wire Wire Line
-	7000 2800 7000 5100
+	7000 2800 7000 3150
 Wire Wire Line
 	7000 5100 5150 5100
@@
 	6700 2700 7100 2700
 Wire Wire Line
-	7100 2700 7100 5200
+	7100 2700 7100 3050
 Wire Wire Line
 	7100 5200 5050 5200
@@
 	5050 4400 4450 4400
 Wire Wire Line
-	6700 2600 7450 2600
+	6700 2600 7200 2600
 Wire Wire Line
 	7200 2600 7200 5250
@@
 	7950 5300 7950 4150
 Wire Wire Line
-	7450 5500 7450 3950
+	7450 5500 7450 4250
 Wire Wire Line
 	7450 3850 7350 3850
@@
 	9650 2950 9850 2950
 Wire Wire Line
-	9850 2950 9850 5300
+	9850 2950 9850 3150
 Wire Wire Line
 	9850 3150 9650 3150
@@
 	5300 4400 5300 5500
 Wire Wire Line
-	2700 5500 7450 5500
+	2700 5500 5300 5500
 Wire Wire Line
 	5300 4000 5100 4000
@@
 Connection ~ 5300 5500
 Connection ~ 7450 4250
+Wire Wire Line
+	1700 5300 1700 5350
+Wire Wire Line
+	1700 3300 1700 3200
+Wire Wire Line
+	1700 3200 1700 2300
+Wire Wire Line
+	1700 3800 1700 3300
+Wire Wire Line
+	1700 4000 1700 3800
+Wire Wire Line
+	2650 2300 3750 2300
+Wire Wire Line
+	2250 5300 1700 5300
+Wire Wire Line
+	3750 5300 2250 5300
+Wire Wire Line
+	3750 2300 5100 2300
+Wire Wire Line
+	7200 2600 7450 2600
+Wire Wire Line
+	7100 3050 7100 5200
+Wire Wire Line
+	7000 3150 7000 5100
+Wire Wire Line
+	6900 3250 6900 4600
+Wire Wire Line
+	6850 3350 6850 4700
+Wire Wire Line
+	6800 3450 6800 4800
+Wire Wire Line
+	6750 3550 6750 4900
+Wire Wire Line
+	6700 3650 6700 5000
+Wire Wire Line
+	9850 3150 9850 3350
+Wire Wire Line
+	9850 3350 9850 3550
+Wire Wire Line
+	9850 3550 9850 3750
+Wire Wire Line
+	9850 3750 9850 3950
+Wire Wire Line
+	9850 3950 9850 4150
+Wire Wire Line
+	9850 4150 9850 4350
+Wire Wire Line
+	7950 5300 6000 5300
+Wire Wire Line
+	9850 4350 9850 5300
+Wire Wire Line
+	6000 5300 3750 5300
+Wire Wire Line
+	6000 2300 7950 2300
+Wire Wire Line
+	5100 2300 6000 2300
+Wire Wire Line
+	5300 5500 7450 5500
+Wire Wire Line
+	7450 4250 7450 3950
 $EndSCHEMATC

Commit message: Save all Schematics again to overcome problems with version change
Parts:
- SW?: symbol switches:SW_SPST -> Z80Rom-rescue:SW_SPST-switches
- U1: symbol Zilog:Z80CPU -> Z80Rom-rescue:Z80CPU-Zilog
- U2: symbol memory:27C64 -> Z80Rom-rescue:27C64-memory
Changed lines of the file:
@@
 $EndDescr
 $Comp
-L Zilog:Z80CPU U1
+L Z80Rom-rescue:Z80CPU-Zilog U1
 U 1 1 5A1A6EC8
 P 3750 3800
@@
 $EndComp
 $Comp
-L switches:SW_SPST SW?
+L Z80Rom-rescue:SW_SPST-switches SW?
 U 1 1 5A1A73BF
 P 2450 2900
@@
 1.0
 $Comp
-L memory:27C64 U2
+L Z80Rom-rescue:27C64-memory U2
 U 1 1 5A1C6F65
 P 6000 3500
