File: Schematics/Z80Test/Z80Test.sch (KiCad schematic (older format))
At the start: 20 parts, among them U1 Z80ACPU

Commit message: Update schematics to KiCad 5
Parts:
- C1: symbol CP1 -> Device:CP1
- D1, D2, D3, D4, D5, D6, D7, D8: symbol LED -> Device:LED
- R1, R2, R3, R4, R5, R6, R7, R8, R9: symbol R -> Device:R
- SW?: symbol SW_SPST -> switches:SW_SPST
- U1: symbol Z80CPU -> Zilog:Z80CPU
Changed lines of the file:
@@
-EESchema Schematic File Version 2
-LIBS:Zilog
-LIBS:power
-LIBS:device
-LIBS:switches
-LIBS:relays
-LIBS:motors
-LIBS:transistors
-LIBS:conn
-LIBS:linear
-LIBS:regul
-LIBS:74xx
-LIBS:cmos4000
-LIBS:adc-dac
-LIBS:memory
-LIBS:xilinx
-LIBS:microcontrollers
-LIBS:dsp
-LIBS:microchip
-LIBS:analog_switches
-LIBS:motorola
-LIBS:texas
-LIBS:intel
-LIBS:audio
-LIBS:interface
-LIBS:digital-audio
-LIBS:philips
-LIBS:display
-LIBS:cypress
-LIBS:siliconi
-LIBS:opto
-LIBS:atmel
-LIBS:contrib
-LIBS:valves
-LIBS:cmos_ieee
+EESchema Schematic File Version 4
 LIBS:Z80Test-cache
-EELAYER 25 0
+EELAYER 26 0
 EELAYER END
 $Descr A4 11693 8268
@@
 $EndDescr
 $Comp
-L Z80CPU U1
+L Zilog:Z80CPU U1
 U 1 1 5A1A6EC8
 P 5600 3850
@@
 $EndComp
 $Comp
-L VCC #PWR?
+L power:VCC #PWR?
 U 1 1 5A1A6F3C
 P 3550 2350
@@
 $EndComp
 $Comp
-L GND #PWR?
+L power:GND #PWR?
 U 1 1 5A1A6F76
 P 3550 5400
@@
 $EndComp
 $Comp
-L CP1 C1
+L Device:CP1 C1
 U 1 1 5A1A6FD7
 P 3550 5050
@@
 $EndComp
 $Comp
-L R R1
+L Device:R R1
 U 1 1 5A1A7360
 P 4500 2650
@@
 $EndComp
 $Comp
-L SW_SPST SW?
+L switches:SW_SPST SW?
 U 1 1 5A1A73BF
 P 4300 2950
@@
 Clock
 $Comp
-L R R2
+L Device:R R2
 U 1 1 5A1A77ED
 P 7150 2650
@@
 $EndComp
 $Comp
-L R R3
+L Device:R R3
 U 1 1 5A1A7868
 P 7150 2850
@@
 $EndComp
 $Comp
-L R R4
+L Device:R R4
 U 1 1 5A1A78C6
 P 7150 3050
@@
 $EndComp
 $Comp
-L R R5
+L Device:R R5
 U 1 1 5A1A78F7
 P 7150 3250
@@
 $EndComp
 $Comp
-L R R6
+L Device:R R6
 U 1 1 5A1A792F
 P 7150 3450
@@
 $EndComp
 $Comp
-L R R7
+L Device:R R7
 U 1 1 5A1A796A
 P 7150 3650
@@
 $EndComp
 $Comp
-L R R8
+L Device:R R8
 U 1 1 5A1A799E
 P 7150 3850
@@
 $EndComp
 $Comp
-L R R9
+L Device:R R9
 U 1 1 5A1A79DB
 P 7150 4050
@@
 $EndComp
 $Comp
-L LED D1
+L Device:LED D1
 U 1 1 5A1A834A
 P 7600 2650
@@
 $EndComp
 $Comp
-L LED D2
+L Device:LED D2
 U 1 1 5A1A8394
 P 7600 2850
@@
 $EndComp
 $Comp
-L LED D3
+L Device:LED D3
 U 1 1 5A1A83D6
 P 7600 3050
@@
 $EndComp
 $Comp
-L LED D4
+L Device:LED D4
 U 1 1 5A1A841B
 P 7600 3250
@@
 $EndComp
 $Comp
-L LED D5
+L Device:LED D5
 U 1 1 5A1A8463
 P 7600 3450
@@
 $EndComp
 $Comp
-L LED D6
+L Device:LED D6
 U 1 1 5A1A84AC
 P 7600 3650
@@
 $EndComp
 $Comp
-L LED D8
+L Device:LED D8
 U 1 1 5A1A854B
 P 7600 4050
@@
 $EndComp
 $Comp
-L LED D7
+L Device:LED D7
 U 1 1 5A1A8B0F
 P 7600 3850
@@
 Connection ~ 3550 2350
 Wire Wire Line
-	7950 5350 3550 5350
-Wire Wire Line
-	3550 5200 3550 5400
+	7950 5350 7250 5350
+Wire Wire Line
+	3550 5200 3550 5350
 Connection ~ 3550 5350
 Wire Wire Line
-	3550 2350 5600 2350
-Wire Wire Line
-	3550 4900 3550 2350
+	3550 2350 4500 2350
+Wire Wire Line
+	3550 4900 3550 4050
 Wire Wire Line
 	4900 3350 3550 3350
@@
 	7750 2650 7950 2650
 Wire Wire Line
-	7950 2650 7950 5350
+	7950 2650 7950 2850
 Wire Wire Line
 	7950 2850 7750 2850
@@
 	6300 4350 7250 4350
 Wire Wire Line
-	7250 4350 7250 5350
+	7250 4350 7250 4450
 Connection ~ 7250 5350
 Wire Wire Line
@@
 	6300 5050 7250 5050
 Connection ~ 7250 5050
+Wire Wire Line
+	3550 5350 3550 5400
+Wire Wire Line
+	3550 3350 3550 3250
+Wire Wire Line
+	3550 3250 3550 2350
+Wire Wire Line
+	3550 3850 3550 3350
+Wire Wire Line
+	3550 4050 3550 3850
+Wire Wire Line
+	4500 2350 5600 2350
+Wire Wire Line
+	4100 5350 3550 5350
+Wire Wire Line
+	5600 5350 4100 5350
+Wire Wire Line
+	7950 2850 7950 3050
+Wire Wire Line
+	7950 3050 7950 3250
+Wire Wire Line
+	7950 3250 7950 3450
+Wire Wire Line
+	7950 3450 7950 3650
+Wire Wire Line
+	7950 3650 7950 3850
+Wire Wire Line
+	7950 3850 7950 4050
+Wire Wire Line
+	7950 4050 7950 5350
+Wire Wire Line
+	7250 5350 5600 5350
+Wire Wire Line
+	7250 4450 7250 4550
+Wire Wire Line
+	7250 4550 7250 4650
+Wire Wire Line
+	7250 4650 7250 4750
+Wire Wire Line
+	7250 4750 7250 4850
+Wire Wire Line
+	7250 4850 7250 4950
+Wire Wire Line
+	7250 4950 7250 5050
+Wire Wire Line
+	7250 5050 7250 5350
 $EndSCHEMATC

Commit message: Save all Schematics again to overcome problems with version change
Parts:
- SW?: symbol switches:SW_SPST -> Z80Test-rescue:SW_SPST-switches
- U1: symbol Zilog:Z80CPU -> Z80Test-rescue:Z80CPU-Zilog
Changed lines of the file:
@@
 $EndDescr
 $Comp
-L Zilog:Z80CPU U1
+L Z80Test-rescue:Z80CPU-Zilog U1
 U 1 1 5A1A6EC8
 P 5600 3850
@@
 $EndComp
 $Comp
-L switches:SW_SPST SW?
+L Z80Test-rescue:SW_SPST-switches SW?
 U 1 1 5A1A73BF
 P 4300 2950
