File: Schematics/SimpleProgrammableClock/SimpleClock.sch (KiCad schematic (older format))
At the start: 8 parts, among them J1 SPI Connector, J2 Rainbow Bus, SW1 SW_Push_Dual, U1 ATmega328-PU

Commit message: Add first revision of keyboard code (arduino mega)
Parts:
- added C2: 100u, Capacitor_THT:CP_Radial_D8.0mm_P3.50mm, symbol Device:CP_Small
- C1: footprint (none) -> Capacitor_THT:C_Disc_D5.1mm_W3.2mm_P5.00mm
- D1: footprint (none) -> Diode_THT:D_DO-15_P12.70mm_Horizontal
- J1: footprint (none) -> Connector_PinHeader_2.54mm:PinHeader_2x05_P2.54mm_Vertical
- J2: footprint (none) -> Connector_PinHeader_2.54mm:PinHeader_1x25_P2.54mm_Vertical
- R1, R2: footprint (none) -> Resistor_THT:R_Axial_DIN0207_L6.3mm_D2.5mm_P10.16mm_Horizontal
- SW1: value SW_Push_Dual -> SW; footprint (none) -> Button_Switch_THT:SW_PUSH_6mm_H4.3mm; symbol Switch:SW_Push_Dual -> Switch:SW_Push
Connections:
- net labels added: +5V, GNDPWR
- wire segments 58 -> 70
- no-connect marks 42 -> 44
Changed lines of the file:
@@
 EESchema Schematic File Version 4
-EELAYER 26 0
+LIBS:SimpleClock-cache
+EELAYER 29 0
 EELAYER END
 $Descr A4 11693 8268
@@
 F 0 "J1" H 3350 3117 50  0000 C CNN
 F 1 "SPI Connector" H 3550 3050 50  0000 C CNN
-F 2 "" H 3300 2700 50  0001 C CNN
+F 2 "Connector_PinHeader_2.54mm:PinHeader_2x05_P2.54mm_Vertical" H 3300 2700 50  0001 C CNN
 F 3 "~" H 3300 2700 50  0001 C CNN
 	1    3300 2700
@@
 	5850 2250 5850 2100
 Wire Wire Line
-	3500 2100 4600 2100
+	3500 2100 3950 2100
 Connection ~ 5750 2100
 Wire Wire Line
 	5750 2100 5850 2100
-Wire Wire Line
-	5750 5250 4650 5250
 Wire Wire Line
 	3850 5250 3850 3300
@@
 F 0 "J2" H 7800 3550 50  0000 L CNN
 F 1 "Rainbow Bus" H 7550 3450 50  0000 L CNN
-F 2 "" H 8250 3300 50  0001 C CNN
+F 2 "Connector_PinHeader_2.54mm:PinHeader_1x25_P2.54mm_Vertical" H 8250 3300 50  0001 C CNN
 F 3 "~" H 8250 3300 50  0001 C CNN
 	1    8250 3300
@@
 $EndComp
 Wire Wire Line
-	8050 2100 5850 2100
+	8050 2100 7450 2100
 Connection ~ 5850 2100
 Wire Wire Line
@@
 Wire Wire Line
 	7200 2300 7200 4300
-Wire Wire Line
-	7200 5250 5750 5250
-Connection ~ 5750 5250
 Wire Wire Line
 	8050 4300 7200 4300
@@
 F 0 "C1" H 4692 2346 50  0000 L CNN
 F 1 "100n" H 4692 2255 50  0000 L CNN
-F 2 "" H 4600 2300 50  0001 C CNN
+F 2 "Capacitor_THT:C_Disc_D5.1mm_W3.2mm_P5.00mm" H 4600 2300 50  0001 C CNN
 F 3 "~" H 4600 2300 50  0001 C CNN
 	1    4600 2300
@@
 	4600 2100 5050 2100
 Wire Wire Line
-	4600 2550 3850 2550
+	4600 2550 3950 2550
 Wire Wire Line
 	3850 2550 3850 2800
@@
 Connection ~ 3850 2800
 $Comp
-L Switch:SW_Push_Dual SW1
+L Switch:SW_Push SW1
 U 1 1 5CB41666
-P 4600 3100
-F 0 "SW1" H 4600 3293 50  0000 C CNN
-F 1 "SW_Push_Dual" H 4600 3294 50  0001 C CNN
-F 2 "" H 4600 3300 50  0001 C CNN
-F 3 "" H 4600 3300 50  0001 C CNN
-	1    4600 3100
-	1    0    0    -1
-$EndComp
-NoConn ~ 4400 3100
-NoConn ~ 4800 3100
+P 4650 3300
+F 0 "SW1" H 4650 3493 50  0000 C CNN
+F 1 "SW" H 4650 3494 50  0001 C CNN
+F 2 "Button_Switch_THT:SW_PUSH_6mm_H4.3mm" H 4650 3500 50  0001 C CNN
+F 3 "" H 4650 3500 50  0001 C CNN
+	1    4650 3300
+	1    0    0    -1
+$EndComp
 $Comp
 L Device:R R1
@@
 F 0 "R1" V 3893 3300 50  0000 C CNN
 F 1 "10k" V 3984 3300 50  0000 C CNN
-F 2 "" V 4030 3300 50  0001 C CNN
+F 2 "Resistor_THT:R_Axial_DIN0207_L6.3mm_D2.5mm_P10.16mm_Horizontal" V 4030 3300 50  0001 C CNN
 F 3 "~" H 4100 3300 50  0001 C CNN
 	1    4100 3300
@@
 $EndComp
 Wire Wire Line
-	4400 3300 4300 3300
-Wire Wire Line
 	3950 3300 3850 3300
 Connection ~ 3850 3300
 Wire Wire Line
 	3850 3300 3850 2800
-Wire Wire Line
-	4800 3300 5050 3300
 Connection ~ 5050 2100
 Wire Wire Line
@@
 F 0 "D1" V 4642 4633 50  0000 R CNN
 F 1 "LED_ALT" V 4597 4632 50  0001 R CNN
-F 2 "" H 4650 4750 50  0001 C CNN
+F 2 "Diode_THT:D_DO-15_P12.70mm_Horizontal" H 4650 4750 50  0001 C CNN
 F 3 "~" H 4650 4750 50  0001 C CNN
 	1    4650 4750
@@
 F 0 "R2" H 4580 4254 50  0000 R CNN
 F 1 "1k" H 4580 4345 50  0000 R CNN
-F 2 "" V 4580 4300 50  0001 C CNN
+F 2 "Resistor_THT:R_Axial_DIN0207_L6.3mm_D2.5mm_P10.16mm_Horizontal" V 4580 4300 50  0001 C CNN
 F 3 "~" H 4650 4300 50  0001 C CNN
 	1    4650 4300
@@
 	5050 3700 5050 3300
 Connection ~ 5050 3300
+$Comp
+L Device:CP_Small C2
+U 1 1 5CB8B6CC
+P 3950 2300
+F 0 "C2" H 4038 2346 50  0000 L CNN
+F 1 "100u" H 4038 2255 50  0000 L CNN
+F 2 "Capacitor_THT:CP_Radial_D8.0mm_P3.50mm" H 3950 2300 50  0001 C CNN
+F 3 "~" H 3950 2300 50  0001 C CNN
+	1    3950 2300
+	1    0    0    -1
+$EndComp
+Wire Wire Line
+	3950 2200 3950 2100
+Connection ~ 3950 2100
+Wire Wire Line
+	3950 2100 4600 2100
+Wire Wire Line
+	3950 2400 3950 2550
+Connection ~ 3950 2550
+Wire Wire Line
+	3950 2550 3850 2550
+Connection ~ 7200 5250
+$Comp
+L power:+5V #PWR0102
+U 1 1 5CB90567
+P 7100 1750
+F 0 "#PWR0102" H 7100 1600 50  0001 C CNN
+F 1 "+5V" H 7115 1923 50  0000 C CNN
+F 2 "" H 7100 1750 50  0001 C CNN
+F 3 "" H 7100 1750 50  0001 C CNN
+	1    7100 1750
+	1    0    0    -1
+$EndComp
+Wire Wire Line
+	7100 1750 7100 2100
+Connection ~ 7100 2100
+Wire Wire Line
+	7100 2100 5850 2100
+NoConn ~ 3500 2900
+NoConn ~ 3500 2700
+NoConn ~ 3500 2600
+NoConn ~ 3000 2600
+$Comp
+L power:PWR_FLAG #FLG0101
+U 1 1 5CB98331
+P 7450 1850
+F 0 "#FLG0101" H 7450 1925 50  0001 C CNN
+F 1 "PWR_FLAG" H 7450 2023 50  0000 C CNN
+F 2 "" H 7450 1850 50  0001 C CNN
+F 3 "~" H 7450 1850 50  0001 C CNN
+	1    7450 1850
+	1    0    0    -1
+$EndComp
+Wire Wire Line
+	7450 1850 7450 2100
+Connection ~ 7450 2100
+Wire Wire Line
+	7450 2100 7100 2100
+$Comp
+L power:GNDPWR #PWR0103
+U 1 1 5CB99EC3
+P 7550 5450
+F 0 "#PWR0103" H 7550 5250 50  0001 C CNN
+F 1 "GNDPWR" H 7554 5296 50  0000 C CNN
+F 2 "" H 7550 5400 50  0001 C CNN
+F 3 "" H 7550 5400 50  0001 C CNN
+	1    7550 5450
+	1    0    0    -1
+$EndComp
+Wire Wire Line
+	7200 5250 7550 5250
+Wire Wire Line
+	7550 5250 7550 5450
+Wire Wire Line
+	4650 5250 5750 5250
+Wire Wire Line
+	5750 5150 5750 5250
+Connection ~ 5750 5250
+Wire Wire Line
+	5750 5250 7200 5250
+$Comp
+L power:PWR_FLAG #FLG0102
+U 1 1 5CBA8643
+P 7550 5000
+F 0 "#FLG0102" H 7550 5075 50  0001 C CNN
+F 1 "PWR_FLAG" H 7550 5173 50  0000 C CNN
+F 2 "" H 7550 5000 50  0001 C CNN
+F 3 "~" H 7550 5000 50  0001 C CNN
+	1    7550 5000
+	1    0    0    -1
+$EndComp
+Wire Wire Line
+	7550 5000 7550 5250
+Connection ~ 7550 5250
+Wire Wire Line
+	4850 3300 5050 3300
+Wire Wire Line
+	4300 3300 4450 3300
 $EndSCHEMATC
